File: 05-adsr-vca/electronics/core/adsr-vca-core.kicad_pcb (KiCad board)
At the start: 2 copper layers, 58 x 65 mm, 68 parts, among them J2 Conn_02x03_Odd_Even, J3 Conn_02x03_Odd_Even, J4 Conn_02x06_Odd_Even, J5 Conn_02x03_Odd_Even, J6 Conn_01x02, J7 Conn_02x05_Odd_Even, J8 Conn_02x03_Odd_Even, Q1 BC857, Q3 BC847BS, U1 LM324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

Commit message: Added VCA amp bias pot
Parts:
- removed R19: 200k, Resistor_SMD:R_0603_1608Metric
Connections:
- C7 pad 1: Net-(U2A--) -> VCA_CV
- R21 pad 1: Net-(U2A--) -> VCA_CV
- R29 pad 2: Net-(U2A--) -> VCA_CV
- U2 pad 2: Net-(U2A--) -> VCA_CV
Routing:
- net VCA_CV: track 4.96 -> 17.8 mm
- net Net-(U2A--): track 11.3 -> 0.00 mm
