File: 05-adsr-vca/electronics/core/sheets/vca.kicad_sch (KiCad schematic)
At the start: 20 parts, among them Q3 BC847BS, U2 TL072

Commit message: Added VCA amp bias pot
Parts:
- removed R19: 200k, Resistor_SMD:R_0603_1608Metric, symbol Device:R
Connections:
- net CV: now also C7.1, R21.1, R29.2, U2.2 (-)
Other:
- note added: "CV inputs can be mixed on the UI board by using 200k input resistors on all inputs."
Changed lines of the file:
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@@
 	(generator_version "9.0")
 	(paper "A4")
+	(text "CV inputs can be mixed on the UI board \nby using 200k input resistors on all inputs."
+		(exclude_from_sim no)
+		(at 39.37 88.9 0)
+		(effects
+			(font
+				(size 1.5 1.5)
+				(thickness 0.1875)
+				(color 255 0 255 1)
+			)
+			(justify left)
+		)
+	)
 	(text "There was a crosstalk issue because\nthe 100k resistor was too far from \nthe input pin header on the PCB. It's\nnow moved as close to it as possible\nso that the input signal is scaled down\ndrastically as it enters the board.\n\nNote that now there's a 100k resistor \non the UI board too for testing purposes. \nEither that OR R18 (on this board) should be \nused, so make sure to short one of them."
 		(exclude_from_sim no)
@@
 	(wire
 		(pts
-			(xy 81.28 110.49) (xy 97.79 110.49)
+			(xy 81.28 110.49) (xy 111.76 110.49)
 		)
 		(stroke
@@
 	(wire
 		(pts
-			(xy 105.41 110.49) (xy 111.76 110.49)
-		)
-		(stroke
-			(width 0)
-			(type default)
-		)
-	)
-	(wire
-		(pts
 			(xy 137.16 58.42) (xy 137.16 66.04)
 		)
@@
 		)
 	)
+	(polyline
+		(pts
+			(xy 80.01 107.95) (xy 80.01 92.71)
+		)
+		(stroke
+			(width 0.5)
+			(type solid)
+			(color 255 0 255 1)
+		)
+	)
 	(wire
 		(pts
@@
 					(unit 1)
 				)
-			)
-		)
-	)
-	(symbol
-		(lib_id "Device:R")
-		(at 101.6 110.49 90)
-		(unit 1)
-		(exclude_from_sim no)
-		(in_bom yes)
-		(on_board yes)
-		(dnp no)
-		(property "Reference" "R19"
-			(at 101.6 104.14 90)
-			(effects
-				(font
-					(size 1.27 1.27)
-				)
-			)
-		)
-		(property "Value" "200k"
-			(at 101.6 106.68 90)
-			(effects
-				(font
-					(size 1.27 1.27)
-				)
-			)
-		)
-		(property "Footprint" "Resistor_SMD:R_0603_1608Metric"
-			(at 101.6 112.268 90)
-			(effects
-				(font
-					(size 1.27 1.27)
-				)
-				(hide yes)
-			)
-		)
-		(property "Datasheet" "~"
-			(at 101.6 110.49 0)
-			(effects
-				(font
-					(size 1.27 1.27)
-				)
-				(hide yes)
-			)
-		)
-		(property "Description" ""
-			(at 101.6 110.49 0)
-			(effects
-				(font
-					(size 1.27 1.27)
-				)
-				(hide yes)
-			)
-		)
-		(property "LCSC" "C25811"
-			(at 101.6 110.49 90)
-			(effects
-				(font
-					(size 1.27 1.27)
-				)
-				(hide yes)
-			)
-		)
-		(property "CHECKED" "YES"
-			(at 101.6 110.49 90)
-			(effects
-				(font
-					(size 1.27 1.27)
-				)
-				(hide yes)
-			)
-		)
-		(property "Vendor" "JLCPCB"
-			(at 101.6 110.49 90)
-			(effects
-				(font
-					(size 1.27 1.27)
-				)
-				(hide yes)
-			)
-		)
-		(property "Part No." ""
-			(at 101.6 110.49 0)
-			(effects
-				(font
-					(size 1.27 1.27)
-				)
-				(hide yes)
-			)
-		)
-		(property "Part URL" ""
-			(at 101.6 110.49 0)
-			(effects
-				(font
-					(size 1.27 1.27)
-				)
-				(hide yes)
-			)
-		)
-		(property "Arwill" ""
-			(at 101.6 110.49 90)
-			(effects
-				(font
-					(size 1.27 1.27)
-				)
-				(hide yes)
-			)
-		)
-		(property "Hestore" ""
-			(at 101.6 110.49 90)
-			(effects
-				(font
-					(size 1.27 1.27)
-				)
-				(hide yes)
-			)
-		)
-		(pin "1"
-		)
-		(pin "2"
-		)
-		(instances
-			(project "adsr-vca-core"
-				(path "/8e2e31f3-eed5-4de1-966c-f4162758c735/c6cac276-2f32-41b3-9c97-03c30aa61119"
-					(reference "R19")
-					(unit 1)
-				)
