File: modules/07-brain/electronics/ui/sheets/leds.kicad_sch (KiCad schematic)
At the start: 24 parts, among them Q1 2N3904, Q2 2N3904, Q3 2N3904, Q4 2N3904, Q5 2N3904, Q6 2N3904

Commit message: Added Brain BOM
Parts:
- Q1, Q2, Q3, Q4, Q5, Q6: Part URL (none) -> https://mou.sr/4febysZ; Part no. (none) -> 637-2N3904; Vendor (none) -> Mouser
- R10, R13, R14, R5, R6, R9: Part URL (none) -> https://mou.sr/4q072Ei; Part no. (none) -> 603-MFR25SFTF52-4K7; Vendor JLCPCB -> Mouser
- R11, R12, R3, R4, R7, R8: Part URL (none) -> https://mou.sr/3MWzgkZ; Part no. (none) -> 603-MFR-25FRF52-47K; Vendor JLCPCB -> Mouser

Commit message: Fixed Brain UI
Parts:
- Q1, Q2, Q3, Q4, Q5, Q6: Part URL https://mou.sr/4febysZ -> (none); Part no. 637-2N3904 -> (none); Vendor Mouser -> (none)
- R10, R13, R14, R5, R6, R9: Part URL https://mou.sr/4q072Ei -> (none); Part no. 603-MFR25SFTF52-4K7 -> (none); Vendor Mouser -> JLCPCB
- R11, R12, R3, R4, R7, R8: Part URL https://mou.sr/3MWzgkZ -> (none); Part no. 603-MFR-25FRF52-47K -> (none); Vendor Mouser -> JLCPCB
