File: modules/02-vco/electronics/ui-glide/vco-ui.kicad_pcb (KiCad board)
At the start: 2 copper layers, 58 x 110 mm, 41 parts, among them J1 Conn_01x04, J2 Conn_02x05_Odd_Even, J3 Conn_02x03_Odd_Even, J4 Conn_01x02, J5 Conn_02x02_Counter_Clockwise, J6 Conn_01x07, U1 0203, U2 TL072

Commit message: Updated glided VCO UI and ADSR UI
Other:
- board text added: "CV OUT"
- board text added: "GLIDE"
- board text removed: "PULSE WIDTH"
Changed lines of the file:
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@@
 		)
 	)
-	(gr_text "PWM"
-		(at 172.768 109.532 0)
+	(gr_text "CV OUT"
+		(at 173.276 106.611 0)
 		(layer "F.SilkS")
 		(effects
@@
 		)
 	)
-	(gr_text "PULSE WIDTH"
+	(gr_text "GLIDE"
 		(at 168.958 93.53 0)
 		(layer "F.SilkS")
