File: modules/01-psu/electronics/moduleur-enclosure/psu.kicad_sch (KiCad schematic)
At the start: 25 parts, among them IC1 ISOLATED_DC-DC_CONV, J1 Barrel_Jack_Switch, J13 Conn_01x03, J2 Conn_02x08_Odd_Even, J3 Conn_02x08_Odd_Even, J4 Conn_02x08_Odd_Even, J5 Conn_02x08_Odd_Even

Commit message: Fixed Moduleur PSU Eurorack connector BOM part no.
ref. https://github.com/shmoergh/moduleur/issues/9
Parts:
- J2, J3, J4, J5: Part No. 737-BHR-16-VUA -> 710-61201621721; Part URL https://mou.sr/4jUmWfT -> https://mou.sr/3MHt28J
Changed lines of the file:
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@@
 			)
 		)
-		(property "Part No." "737-BHR-16-VUA"
+		(property "Part No." "710-61201621721 "
 			(at 120.65 138.43 0)
 			(effects
@@
 			)
 		)
-		(property "Part URL" "https://mou.sr/4jUmWfT"
+		(property "Part URL" "https://mou.sr/3MHt28J"
 			(at 120.65 138.43 0)
 			(effects
@@
 			)
 		)
-		(property "Part No." "737-BHR-16-VUA"
+		(property "Part No." "710-61201621721 "
 			(at 186.69 138.43 0)
 			(effects
@@
 			)
 		)
-		(property "Part URL" "https://mou.sr/4jUmWfT"
+		(property "Part URL" "https://mou.sr/3MHt28J"
 			(at 186.69 138.43 0)
 			(effects
@@
 			)
 		)
-		(property "Part No." "737-BHR-16-VUA"
+		(property "Part No." "710-61201621721 "
 			(at 153.67 138.43 0)
 			(effects
@@
 			)
 		)
-		(property "Part URL" "https://mou.sr/4jUmWfT"
+		(property "Part URL" "https://mou.sr/3MHt28J"
 			(at 153.67 138.43 0)
 			(effects
@@
 			)
 		)
-		(property "Part No." "737-BHR-16-VUA"
+		(property "Part No." "710-61201621721 "
 			(at 86.36 138.43 0)
 			(effects
@@
 			)
 		)
-		(property "Part URL" "https://mou.sr/4jUmWfT"
+		(property "Part URL" "https://mou.sr/3MHt28J"
 			(at 86.36 138.43 0)
 			(effects
