File: modules/01-psu/electronics/moduleur-enclosure/psu.kicad_pcb (KiCad board)
At the start: 2 copper layers, 250 x 32 mm, 32 parts, among them IC1 ISOLATED_DC-DC_CONV, J1 Barrel_Jack_Switch, J13 Conn_01x03, J2 Conn_02x08_Odd_Even, J3 Conn_02x08_Odd_Even, J4 Conn_02x08_Odd_Even, J5 Conn_02x08_Odd_Even

Commit message: PSU/Moduleur ready for v1.0
Other:
- board text added: "POWER SUPPLY (V1.0)"
- board text removed: "POWER SUPPLY (V0.2)"
Changed lines of the file:
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@@
 		)
 		(fp_text user "${REFERENCE}"
-			(at 8.83 -8.89 180)
+			(at 8.83 -8.89 0)
 			(layer "B.Fab")
 			(effects
@@
 		)
 	)
-	(gr_text "POWER SUPPLY (V0.2)"
+	(gr_text "POWER SUPPLY (V1.0)"
 		(at 39.116 80.518 90)
 		(layer "B.SilkS")
@@
 			(justify left bottom mirror)
 		)
-		(render_cache "POWER SUPPLY (V0.2)" 90
+		(render_cache "POWER SUPPLY (V1.0)" 90
 			(polygon
 				(pts
@@
 			(polygon
 				(pts
-					(xy 37.518824 100.734346) (xy 38.670124 100.734346) (xy 38.670124 100.931084) (xy 38.288281 100.931084)
-					(xy 38.288281 101.122051) (xy 38.091543 101.122051) (xy 38.091543 100.931084) (xy 37.518824 100.931084)
-				)
-			)
-			(polygon
-				(pts
-					(xy 38.664262 100.925222) (xy 38.861 100.925222) (xy 38.861 101.503803) (xy 38.664262 101.503803)
-				)
-			)
-			(polygon
-				(pts
-					(xy 37.327857 100.925222) (xy 37.524686 100.925222) (xy 37.524686 101.503803) (xy 37.327857 101.503803)
-				)
-			)
-			(polygon
-				(pts
-					(xy 37.518824 101.497941) (xy 37.7097 101.497941) (xy 37.7097 101.307065) (xy 37.906529 101.307065)
-					(xy 37.906529 101.497941) (xy 38.670124 101.497941) (xy 38.670124 101.69477) (xy 37.518824 101.69477)
-				)
-			)
-			(polygon
-				(pts
-					(xy 37.900667 101.116189) (xy 38.097405 101.116189) (xy 38.097405 101.312927) (xy 37.900667 101.312927)
+					(xy 37.715562 101.116189) (xy 38.664262 101.116189) (xy 38.664262 100.734346) (xy 38.861 100.734346)
+					(xy 38.861 101.69477) (xy 38.664262 101.69477) (xy 38.664262 101.312927) (xy 37.327857 101.312927)
+					(xy 37.327857 101.116189) (xy 37.518824 101.116189) (xy 37.518824 100.734346) (xy 37.715562 100.734346)
 				)
 			)
@@
 			(polygon
 				(pts
-					(xy 38.473386 103.404409) (xy 38.861 103.404409) (xy 38.861 104.364833) (xy 38.664262 104.364833)
-					(xy 38.664262 103.601147) (xy 38.473386 103.601147)
-				)
-			)
-			(polygon
-				(pts
-					(xy 37.524686 104.173866) (xy 37.327857 104.173866) (xy 37.327857 103.595285) (xy 37.524686 103.595285)
-				)
-			)
-			(polygon
-				(pts
-					(xy 37.518824 104.168004) (xy 37.906529 104.168004) (xy 37.906529 104.364833) (xy 37.518824 104.364833)
-				)
-			)
-			(polygon
-				(pts
-					(xy 38.282419 103.595285) (xy 38.479248 103.595285) (xy 38.479248 103.792114) (xy 38.282419 103.792114)
-				)
-			)
-			(polygon
-				(pts
-					(xy 37.518824 103.404409) (xy 37.715562 103.404409) (xy 37.715562 103.601147) (xy 37.518824 103.601147)
-				)
-			)
-			(polygon
-				(pts
-					(xy 37.900667 103.977128) (xy 38.097405 103.977128) (xy 38.097405 104.173866) (xy 37.900667 104.173866)
-				)
-			)
-			(polygon
-				(pts
-					(xy 38.091543 103.786252) (xy 38.288281 103.786252) (xy 38.288281 103.98299) (xy 38.091543 103.98299)
-				)
-			)
+					(xy 37.518824 103.404409) (xy 38.670124 103.404409) (xy 38.670124 103.601147) (xy 38.288281 103.601147)
+					(xy 38.288281 103.792114) (xy 38.091543 103.792114) (xy 38.091543 103.601147) (xy 37.518824 103.601147)
+				)
+			)
+			(polygon
+				(pts
+					(xy 38.664262 103.595285) (xy 38.861 103.595285) (xy 38.861 104.173866) (xy 38.664262 104.173866)
+				)
+			)
+			(polygon
+				(pts
+					(xy 37.327857 103.595285) (xy 37.524686 103.595285) (xy 37.524686 104.173866) (xy 37.327857 104.173866)
+				)
+			)
+			(polygon
+				(pts
+					(xy 37.518824 104.168004) (xy 37.7097 104.168004) (xy 37.7097 103.977128) (xy 37.906529 103.977128)
+					(xy 37.906529 104.168004) (xy 38.670124 104.168004) (xy 38.670124 104.364833) (xy 37.518824 104.364833)
+				)
+			)
+			(polygon
+				(pts
+					(xy 37.900667 103.786252) (xy 38.097405 103.786252) (xy 38.097405 103.98299) (xy 37.900667 103.98299)
+				)
+			)
