File: modules/04-vcf/electronics/core/sheets/power.kicad_sch (KiCad schematic)
At the start: 7 parts, among them J6 Conn_02x03_Odd_Even, J7 Conn_01x02, J8 Conn_02x05_Odd_Even

Commit message: Added VCF full BOM
Parts:
- J6, J7, J8: CHECKED (none) -> YES
Changed lines of the file:
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@@
 			)
 		)
-		(property "CHECKED" ""
+		(property "CHECKED" "YES"
 			(at 77.47 87.63 0)
 			(effects
@@
 			)
 		)
-		(property "CHECKED" ""
+		(property "CHECKED" "YES"
 			(at 144.78 92.71 0)
 			(effects
@@
 			)
 		)
-		(property "CHECKED" ""
+		(property "CHECKED" "YES"
 			(at 81.28 104.14 0)
 			(effects

Commit message: Updated out-of-stock 100uF cap JLCPCB product no's
Parts:
- C21, C22: LCSC C2836437 -> C2836442
Changed lines of the file:
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@@
 			)
 		)
-		(property "LCSC" "C2836437"
+		(property "LCSC" "C2836442"
 			(at 219.71 86.36 0)
 			(effects
@@
 			)
 		)
-		(property "LCSC" "C2836437"
+		(property "LCSC" "C2836442"
 			(at 219.71 93.98 0)
 			(effects
