File: modules/04-vcf/electronics/core/sheets/vcf.kicad_sch (KiCad schematic)
At the start: 75 parts, among them J4 S1711-46R, J5 S1711-46R, Q1 BC847BS, U1 TL072, U2 TL072, U3 TL072, U4 TL072

Commit message: VCF JLCPCB verified for v1.0
Parts:
- C10, C12, C14, C18, C19, J4, J5, RV_BALANCE1, RV_MAX_RESO1: CHECKED YES -> (none)
- R13, R22: CHECKED (none) -> YES; LCSC (none) -> C22843; Vendor (none) -> JLCPCB
Other:
- company: (none) -> Shmøergh
- title: (none) -> Steiner-Parker VCF
Changed lines of the file:
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@@
 	(generator_version "9.0")
 	(paper "User" 350 210)
+	(title_block
+		(title "Steiner-Parker VCF")
+		(date "2025-12-11")
+		(company "Shmøergh")
+	)
 	(rectangle
 		(start 125.73 162.56)
@@
 			)
 		)
-		(property "CHECKED" "YES"
+		(property "CHECKED" ""
 			(at 156.21 74.93 0)
 			(effects
@@
 			)
 		)
-		(property "CHECKED" "YES"
+		(property "CHECKED" ""
 			(at 171.45 74.93 0)
 			(effects
@@
 			)
 		)
-		(property "CHECKED" "YES"
+		(property "CHECKED" ""
 			(at 186.69 74.93 0)
 			(effects
@@
 			)
 		)
-		(property "LCSC" ""
+		(property "LCSC" "C22843"
 			(at 133.35 53.34 0)
 			(effects
@@
 			)
 		)
-		(property "Vendor" ""
+		(property "Vendor" "JLCPCB"
 			(at 133.35 53.34 0)
 			(effects
@@
 			)
 		)
-		(property "CHECKED" ""
+		(property "CHECKED" "YES"
 			(at 133.35 53.34 0)
 			(effects
@@
 			)
 		)
-		(property "LCSC" ""
+		(property "LCSC" "C22843"
 			(at 209.55 53.34 0)
 			(effects
@@
 			)
 		)
-		(property "Vendor" ""
+		(property "Vendor" "JLCPCB"
 			(at 209.55 53.34 0)
 			(effects
@@
 			)
 		)
-		(property "CHECKED" ""
+		(property "CHECKED" "YES"
 			(at 209.55 53.34 0)
 			(effects
@@
 			)
 		)
-		(property "CHECKED" "YES"
+		(property "CHECKED" ""
 			(at 224.79 59.69 90)
 			(effects
@@
 			)
 		)
-		(property "CHECKED" "YES"
+		(property "CHECKED" ""
 			(at 271.78 57.15 90)
 			(effects
@@
 			)
 		)
-		(property "CHECKED" "YES"
+		(property "CHECKED" ""
 			(at 171.45 46.99 90)
 			(effects
@@
 			)
 		)
-		(property "CHECKED" "YES"
+		(property "CHECKED" ""
 			(at 264.16 71.12 0)
 			(effects
@@
 			)
 		)
-		(property "CHECKED" "YES"
+		(property "CHECKED" ""
 			(at 252.73 146.05 0)
 			(effects
@@
 			)
 		)
-		(property "CHECKED" "YES"
+		(property "CHECKED" ""
 			(at 252.73 139.7 0)
 			(effects

Commit message: Added VCF full BOM
Parts:
- C10, C12, C14, J4, J5, RV_BALANCE1: CHECKED (none) -> YES
- C18: CHECKED (none) -> YES; Part URL https://mou.sr/4g5F5Xb -> https://mou.sr/48MjAbl; Part no. 80-R82EC1470DQ50K -> 80-R82CC4100AA60J
- C19: CHECKED (none) -> YES; Part URL https://mou.sr/472flJF -> https://mou.sr/455uZSu; Part no. 667-EEA-GA1V470B -> 80-ESK475M035AC3AA
- RV_MAX_RESO1: CHECKED (none) -> YES; Part URL https://mou.sr/3OVlmh2 -> https://mou.sr/4oMQfnb; Part no. 531-PT6KH104A1010PM -> 774-06TR4AA104CP
Changed lines of the file:
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@@
 			)
 		)
-		(property "CHECKED" ""
+		(property "CHECKED" "YES"
 			(at 156.21 74.93 0)
 			(effects
@@
 			)
 		)
-		(property "CHECKED" ""
+		(property "CHECKED" "YES"
 			(at 171.45 74.93 0)
 			(effects
@@
 			)
 		)
-		(property "CHECKED" ""
+		(property "CHECKED" "YES"
 			(at 186.69 74.93 0)
 			(effects
@@
 			)
 		)
-		(property "Part URL" "https://mou.sr/4g5F5Xb"
+		(property "Part URL" "https://mou.sr/48MjAbl"
 			(at 224.79 59.69 0)
 			(effects
@@
 			)
 		)
-		(property "Part no." "80-R82EC1470DQ50K "
+		(property "Part no." "80-R82CC4100AA60J "
 			(at 224.79 59.69 90)
 			(effects
@@
 			)
 		)
-		(property "CHECKED" ""
+		(property "CHECKED" "YES"
 			(at 224.79 59.69 90)
 			(effects
@@
 			)
 		)
-		(property "Part URL" "https://mou.sr/472flJF"
+		(property "Part URL" "https://mou.sr/455uZSu"
 			(at 271.78 57.15 0)
 			(effects
@@
 			)
 		)
-		(property "Part no." "667-EEA-GA1V470B "
+		(property "Part no." "80-ESK475M035AC3AA "
 			(at 271.78 57.15 90)
 			(effects
@@
 			)
 		)
-		(property "CHECKED" ""
+		(property "CHECKED" "YES"
 			(at 271.78 57.15 90)
 			(effects
@@
 			)
 		)
-		(property "CHECKED" ""
+		(property "CHECKED" "YES"
 			(at 171.45 46.99 90)
 			(effects
@@
 			)
 		)
-		(property "Part URL" "https://mou.sr/3OVlmh2"
+		(property "Part URL" "https://mou.sr/4oMQfnb"
 			(at 264.16 71.12 0)
 			(effects
@@
 			)
 		)
-		(property "Part no." "531-PT6KH104A1010PM "
+		(property "Part no." "774-06TR4AA104CP"
 			(at 264.16 71.12 0)
 			(effects
@@
 			)
 		)
-		(property "CHECKED" ""
+		(property "CHECKED" "YES"
 			(at 264.16 71.12 0)
 			(effects
@@
 			)
 		)
-		(property "CHECKED" ""
+		(property "CHECKED" "YES"
 			(at 252.73 146.05 0)
 			(effects
@@
 			)
 		)
-		(property "CHECKED" ""
+		(property "CHECKED" "YES"
 			(at 252.73 139.7 0)
 			(effects

Commit message: Updated out-of-stock 100uF cap JLCPCB product no's
Parts:
- C13, C17: LCSC C2836437 -> C2836442
Changed lines of the file:
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@@
 			)
 		)
-		(property "LCSC" "C2836437"
+		(property "LCSC" "C2836442"
 			(at 181.61 35.56 0)
 			(effects
@@
 			)
 		)
-		(property "LCSC" "C2836437"
+		(property "LCSC" "C2836442"
 			(at 198.12 142.24 0)
 			(effects

Commit message: Updated readme
Other:
- title: Steiner-Parker VCF -> Diode VCF
- moved on the sheet: C16, C17
Changed lines of the file:
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@@
 	(paper "User" 350 210)
 	(title_block
-		(title "Steiner-Parker VCF")
+		(title "Diode VCF")
 		(date "2025-12-11")
 		(company "Shmøergh")
@@
 		)
 	)
+	(rectangle
+		(start 152.4 105.41)
+		(end 191.77 125.73)
+		(stroke
+			(width 0)
+			(type dash)
+		)
+		(fill
+			(type none)
+		)
+	)
 	(text "R3 and R4 only if necessary."
 		(exclude_from_sim no)
@@
 	)
 	(junction
-		(at 181.61 31.75)
-		(diameter 0)
-		(color 0 0 0 0)
-	)
-	(junction
 		(at 171.45 41.91)
 		(diameter 0)
@@
 	)
 	(junction
-		(at 237.49 146.05)
+		(at 166.37 137.16)
 		(diameter 0)
 		(color 0 0 0 0)
 	)
 	(junction
-		(at 240.03 54.61)
+		(at 237.49 146.05)
 		(diameter 0)
 		(color 0 0 0 0)
 	)
 	(junction
-		(at 187.96 137.16)
+		(at 240.03 54.61)
 		(diameter 0)
 		(color 0 0 0 0)
@@
 	(wire
 		(pts
+			(xy 149.86 19.05) (xy 163.83 19.05)
+		)
+		(stroke
+			(width 0)
+			(type default)
+		)
+	)
+	(wire
+		(pts
 			(xy 167.64 46.99) (xy 133.35 46.99)
 		)
@@
 		)
 	)
+	(wire
+		(pts
+			(xy 156.21 137.16) (xy 166.37 137.16)
+		)
+		(stroke
+			(width 0)
+			(type default)
+		)
+	)
 	(polyline
 		(pts
@@
 	(wire
 		(pts
+			(xy 163.83 31.75) (xy 171.45 31.75)
+		)
+		(stroke
+			(width 0)
+			(type default)
+		)
+	)
+	(wire
+		(pts
 			(xy 48.26 63.5) (xy 45.72 63.5)
 		)
@@
 	(wire
 		(pts
-			(xy 180.34 123.19) (xy 180.34 120.65)
+			(xy 163.83 19.05) (xy 163.83 31.75)
 		)
 		(stroke
@@
 	(wire
 		(pts
-			(xy 66.04 60.96) (xy 63.5 60.96)
+			(xy 180.34 123.19) (xy 180.34 120.65)
 		)
 		(stroke
@@
 	(wire
 		(pts
-			(xy 198.12 137.16) (xy 187.96 137.16)
+			(xy 66.04 60.96) (xy 63.5 60.96)
 		)
 		(stroke
@@
 	(wire
 		(pts
-			(xy 181.61 31.75) (xy 193.04 31.75)
+			(xy 293.37 96.52) (xy 297.18 96.52)
 		)
 		(stroke
@@
 	(wire
 		(pts
-			(xy 293.37 96.52) (xy 297.18 96.52)
+			(xy 149.86 21.59) (xy 149.86 19.05)
 		)
 		(stroke
@@
 	(wire
 		(pts
-			(xy 198.12 138.43) (xy 198.12 137.16)
+			(xy 156.21 138.43) (xy 156.21 137.16)
 		)
 		(stroke
@@
 	(symbol
 		(lib_id "power:GND")
-		(at 198.12 146.05 0)
+		(at 156.21 146.05 0)
 		(unit 1)
 		(exclude_from_sim no)
@@
 		(dnp no)
 		(property "Reference" "#PWR022"
-			(at 198.12 152.4 0)
+			(at 156.21 152.4 0)
 			(effects
 				(font
@@
 		)
 		(property "Value" "GND"
-			(at 198.247 150.4442 0)
+			(at 156.337 150.4442 0)
 			(effects
 				(font
@@
 		)
 		(property "Footprint" ""
-			(at 198.12 146.05 0)
+			(at 156.21 146.05 0)
 			(effects
 				(font
@@
 		)
 		(property "Datasheet" ""
-			(at 198.12 146.05 0)
+			(at 156.21 146.05 0)
 			(effects
 				(font
@@
 		)
 		(property "Description" "Power symbol creates a global label with name \"GND\" , ground"
-			(at 198.12 146.05 0)
+			(at 156.21 146.05 0)
 			(effects
 				(font
@@
 	(symbol
 		(lib_id "power:GND")
-		(at 193.04 39.37 0)
+		(at 149.86 29.21 0)
 		(unit 1)
 		(exclude_from_sim no)
@@
 		(dnp no)
 		(property "Reference" "#PWR021"
-			(at 193.04 45.72 0)
+			(at 149.86 35.56 0)
 			(effects
 				(font
@@
 		)
 		(property "Value" "GND"
-			(at 193.167 43.7642 0)
+			(at 149.987 33.6042 0)
 			(effects
 				(font
@@
 		)
 		(property "Footprint" ""
-			(at 193.04 39.37 0)
+			(at 149.86 29.21 0)
 			(effects
 				(font
@@
 		)
 		(property "Datasheet" ""
-			(at 193.04 39.37 0)
+			(at 149.86 29.21 0)
 			(effects
 				(font
@@
 		)
 		(property "Description" "Power symbol creates a global label with name \"GND\" , ground"
-			(at 193.04 39.37 0)
+			(at 149.86 29.21 0)
 			(effects
 				(font
@@
 	(symbol
 		(lib_id "Device:C")
-		(at 193.04 35.56 0)
+		(at 149.86 25.4 0)
 		(unit 1)
 		(exclude_from_sim no)
@@
 		(dnp no)
 		(property "Reference" "C16"
-			(at 195.961 34.3916 0)
+			(at 152.781 24.2316 0)
 			(effects
 				(font
@@
 		)
 		(property "Value" "100n"
-			(at 195.961 36.703 0)
+			(at 152.781 26.543 0)
 			(effects
 				(font
@@
 		)
 		(property "Footprint" "Capacitor_SMD:C_0603_1608Metric"
-			(at 194.0052 39.37 0)
+			(at 150.8252 29.21 0)
 			(effects
 				(font
@@
 		)
 		(property "Datasheet" "~"
-			(at 193.04 35.56 0)
+			(at 149.86 25.4 0)
 			(effects
 				(font
@@
 		)
 		(property "Description" ""
-			(at 193.04 35.56 0)
+			(at 149.86 25.4 0)
 			(effects
 				(font
@@
 		)
 		(property "LCSC" "C14663"
-			(at 193.04 35.56 0)
+			(at 149.86 25.4 0)
 			(effects
 				(font
@@
 		)
 		(property "Part URL" ""
-			(at 193.04 35.56 0)
+			(at 149.86 25.4 0)
 			(effects
 				(font
@@
 		)
 		(property "Vendor" "JLCPCB"
-			(at 193.04 35.56 0)
+			(at 149.86 25.4 0)
 			(effects
 				(font
@@
 		)
 		(property "Arwill" ""
-			(at 193.04 35.56 0)
+			(at 149.86 25.4 0)
 			(effects
 				(font
@@
 		)
 		(property "Hestore" ""
-			(at 193.04 35.56 0)
+			(at 149.86 25.4 0)
 			(effects
 				(font
@@
 		)
 		(property "CHECKED" "YES"
-			(at 193.04 35.56 0)
+			(at 149.86 25.4 0)
 			(effects
 				(font
@@
 	(symbol
 		(lib_id "Device:C_Polarized")
-		(at 198.12 142.24 180)
+		(at 156.21 142.24 0)
+		(mirror x)
 		(unit 1)
 		(exclude_from_sim no)
@@
 		(on_board yes)
 		(dnp no)
-		(fields_autoplaced yes)
 		(property "Reference" "C17"
-			(at 201.93 141.859 0)
+			(at 152.4 141.859 0)
 			(effects
 				(font
@@
 		)
 		(property "Value" "100u"
-			(at 201.93 144.399 0)
+			(at 152.4 144.399 0)
 			(effects
 				(font
@@
 		)
 		(property "Footprint" "Capacitor_SMD:CP_Elec_6.3x7.7"
-			(at 197.1548 138.43 0)
+			(at 157.1752 138.43 0)
 			(effects
 				(font
@@
 		)
 		(property "Datasheet" "~"
-			(at 198.12 142.24 0)
+			(at 156.21 142.24 0)
 			(effects
 				(font
@@
 		)
 		(property "Description" ""
-			(at 198.12 142.24 0)
+			(at 156.21 142.24 0)
 			(effects
 				(font
@@
 		)
 		(property "Part URL" ""
-			(at 198.12 142.24 0)
+			(at 156.21 142.24 0)
 			(effects
 				(font
@@
 		)
 		(property "Vendor" "JLCPCB"
-			(at 198.12 142.24 0)
+			(at 156.21 142.24 0)
 			(effects
 				(font
@@
 		)
 		(property "LCSC" "C2836442"
-			(at 198.12 142.24 0)
+			(at 156.21 142.24 0)
 			(effects
 				(font
@@
 		)
 		(property "FT Rotation Offset" "180"
-			(at 198.12 142.24 0)
+			(at 156.21 142.24 0)
 			(effects
 				(font
@@
 		)
 		(property "Arwill" ""
-			(at 198.12 142.24 0)
+			(at 156.21 142.24 0)
 			(effects
 				(font
@@
 		)
 		(property "Hestore" ""
-			(at 198.12 142.24 0)
+			(at 156.21 142.24 0)
 			(effects
 				(font
@@
 		)
 		(property "CHECKED" "YES"
-			(at 198.12 142.24 0)
+			(at 156.21 142.24 0)
 			(effects
 				(font

Commit message: KiCAD version update - VCF
Other:
- title: Diode VCF -> Moduleur VCF
Changed lines of the file:
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@@
 	(paper "User" 350 210)
 	(title_block
-		(title "Diode VCF")
-		(date "2025-12-11")
+		(title "Moduleur VCF")
+		(date "2026-02-21")
+		(rev "v1.0")
 		(company "Shmøergh")
 	)

Commit message: Cleanup
Connections:
- net CV_I: now reaches Q1.2 (B1), R12.1, R14.1, U2.7
- net FEEDBACK: now reaches C10.2, C14.2, R23.2
- net D_OUT: now reaches C12.1, C18.2, D5.2 (A), D6.1 (K)
- net HP_I: now reaches C12.2, R15.2, R19.1
- net LP_I: now reaches C11.1, R18.2, RV_BALANCE1.2
Other:
- note added: "Diode filter network"
- note removed: "ALL OPAMP POLARITY DOUBLECHECKED"
- note removed: "CHECKED"
- note removed: "Diode network is prone to picking up hum. Must be shielded."
- note removed: "TEST: I never really needed RV_BALANCE1. What if R13 and R22 are 2k and we don't use the trimmer at all (ie. 1,2,3 legs are all connected)? Once tested, R13 and R22 can be SMDs. -> result: WORKS but better to doublecheck again on another test"
- moved on the sheet: C1, C10, C11, C12, C13, C14, C15, C16, C17, C18, C19, C2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

Commit message: Fixed VCF Core schemo and PCB after fckckin KiCAD update
Parts:
- Q1: footprint Package_TO_SOT_SMD:SOT-363_SC-70-6 -> Shmoergh_Custom_Footprints:SOT-363_SC-70-6
