File: enclosure/fr4-enclosure/front/fr4-modular-enclosure-front.kicad_sch (KiCad schematic)
At the start: 0 parts

Commit message: Fixed FR4 enclosure panels
There was an inconsistent behavior on the gerber viewer of JLCPCB. Added a layer of GND to all panels with a plated mounting hole that allows full isolation (Faraday-cage) of the enclosure, to minimize noise.
Parts:
- added H1, H2: MountingHole_Pad, MountingHole:MountingHole_3.2mm_M3_DIN965_Pad_TopOnly, symbol Mechanical:MountingHole_Pad
Connections:
- new net GND: H1.1, H2.1
