File: modules/05-adsr-vca/next/ui/adsr-vca-ui.kicad_sch (KiCad schematic)
At the start: 28 parts, among them J1 Conn_02x03_Odd_Even, J2 Conn_01x02, J3 Conn_01x02, J4 Conn_02x02_Odd_Even, J5 Conn_02x03_Odd_Even, J6 Conn_02x02_Odd_Even, J7 Conn_02x05_Odd_Even, J8 Conn_02x03_Odd_Even

Commit message: Updated mounting hole H3 on Brain to be grounded
Parts:
- removed D7: 1N4148, Diode_THT:D_DO-35_SOD27_P7.62mm_Horizontal, symbol Diode:1N4148
- removed J3: Conn_01x02, Connector_PinSocket_2.54mm:PinSocket_1x02_P2.54mm_Vertical, symbol Connector_Generic:Conn_01x02
- removed J4, J6: Conn_02x02_Odd_Even, Connector_PinSocket_2.54mm:PinSocket_2x02_P2.54mm_Vertical, symbol Connector_Generic:Conn_02x02_Odd_Even
- removed J5: Conn_02x03_Odd_Even, Connector_PinSocket_2.54mm:PinSocket_2x03_P2.54mm_Vertical, symbol Connector_Generic:Conn_02x03_Odd_Even
- removed J7: Conn_02x05_Odd_Even, Connector_PinSocket_2.54mm:PinSocket_2x05_P2.54mm_Vertical, symbol Connector_Generic:Conn_02x05_Odd_Even
- removed J_AUDIO_CV_IN1, J_AUDIO_CV_IN2, J_AUDIO_CV_OUT1, J_AUDIO_CV_OUT2, J_PULSE_IN1, J_PULSE_OUT1: PJ398SM, Shmoergh_Custom_Footprints:Jack_3.5mm_QingPu_WQP-PJ398SM_Vertical_CircularHoles, symbol Shmoergh-Custom-Components:AudioJack2_Thonkiconn_S
- removed R15: 0, Shmoergh_Custom_Footprints:R_Axial_DIN0207_L6.3mm_D2.5mm_P7.62mm_Horizontal, symbol Device:R
- removed RV_POT2, RV_POT3: 100k, Shmoergh_Custom_Footprints:Potentiometer_Bourns_Single-PTV09A, symbol Device:R_Potentiometer
- removed U_BTN1: SW_SPST_Push_LED, Shmoergh_Custom_Footprints:SPST_Circular_Pushbutton_LED, symbol Shmoergh-Custom-Components:SW_SPST_Push_LED
- removed U_BTN2: SW_SPST_Push, Shmoergh_Custom_Footprints:SPST_Circular_Pushbutton_LED, symbol Shmoergh-Custom-Components:SW_SPST_Push_LED
- added C1: 100nF, Capacitor_THT:C_Rect_L7.2mm_W2.5mm_P5.00mm_FKS2_FKP2_MKS2_MKP2, symbol Device:C
- added D1: Red LED, LED_THT:LED_D3.0mm, symbol Device:LED
- added H5, H6: MountingHole, MountingHole:MountingHole_3.2mm_M3_DIN965_Pad, symbol Mechanical:MountingHole
- added J3, J6: Conn_02x03_Odd_Even, Connector_PinSocket_2.54mm:PinSocket_2x03_P2.54mm_Vertical, symbol Connector_Generic:Conn_02x03_Odd_Even
- added J5: Conn_01x06, Connector_PinSocket_2.54mm:PinSocket_1x06_P2.54mm_Vertical, symbol Connector_Generic:Conn_01x06
- added JP_DEFAULT_ENV_TO_VCA1: Jumper_2_Open, Connector_PinHeader_2.54mm:PinHeader_1x02_P2.54mm_Horizontal, symbol Jumper:Jumper_2_Open
- added J_ENV_OUT1, J_VCA_CV1, J_VCA_IN1, J_VCA_OUT1: PJ398SM, Shmoergh_Custom_Footprints:Jack_3.5mm_QingPu_WQP-PJ398SM_Vertical_CircularHoles, symbol Shmoergh-Custom-Components:AudioJack2_Thonkiconn_S
- added Q1: 2N3904, Package_TO_SOT_THT:TO-92_Inline_Wide, symbol Transistor_BJT:2N3904
- added Q2: 2N3906, Package_TO_SOT_THT:TO-92_Inline_Wide, symbol Transistor_BJT:2N3906
- added R3: 4.7k, Shmoergh_Custom_Footprints:R_Axial_DIN0207_L6.3mm_D2.5mm_P7.62mm_Horizontal, symbol Device:R
- added R4: 200k, Shmoergh_Custom_Footprints:R_Axial_DIN0207_L6.3mm_D2.5mm_P7.62mm_Horizontal, symbol Device:R
- added R5: 10k, Shmoergh_Custom_Footprints:R_Axial_DIN0207_L6.3mm_D2.5mm_P7.62mm_Horizontal, symbol Device:R
- added R6: 0, Shmoergh_Custom_Footprints:R_Axial_DIN0207_L6.3mm_D2.5mm_P7.62mm_Horizontal, symbol Device:R
- added RV_DECAY1, RV_RELEASE1: A200k-1M, Shmoergh_Custom_Footprints:Potentiometer_Bourns_Single-PTV09A, symbol Device:R_Potentiometer
- added RV_SUSTAIN1: 10k, PTA4543-2015DPB103:TRIM_PTA4543-2015DPB103, symbol Device:R_Potentiometer
- H3: symbol Mechanical:MountingHole_Pad -> Mechanical:MountingHole
- J_GATE1: renamed from J_MIDI1; value PJ366ST -> PJ398SM; Part no. PJ366ST Stereo -> PJ398SM
- R1: value 1k -> 0; Part URL https://mou.sr/4afrY5O -> https://mou.sr/4hEwI4G; Part no. 603-MFR-25FRE52-1K -> 603-MFR-25FRF52100K
- R2: value 10k -> 47k; Part URL https://mou.sr/4po4TSn -> https://mou.sr/3MWzgkZ; Part no. 603-MFR25SFTF52-10K -> 603-MFR-25FRF52-47K
- RV_ATTACK1: renamed from RV_POT1; value 100k -> A200k-1M; Note Knurled Shaft -> D-Shaft; Part URL https://mou.sr/41lYe2k -> https://mou.sr/3VpxrOs; Part no. 652-PTV09A4025UB104 -> 652-PTV09A4025FA105
- renumbered J2 to J4
Connections:
- net AUDIO_CV_OUT_2 is gone; now on net ATTACK_3: J8.2 (Pin_2)
- net POT_1 is gone; now on net ATTACK_3: RV_ATTACK1.2
- net +12V: now also R3.1
- net -12V: now also Q2.3 (C)
- net GND: now also C1.2, J_ENV_OUT1.S, J_VCA_CV1.S, J_VCA_IN1.S, J_VCA_OUT1.S, Q2.2 (B); no longer H3.1, J8.1 (Pin_1), J8.3 (Pin_3), J8.4 (Pin_4), J8.6 (Pin_6), R2.1, RV_ATTACK1.1
- net VCA_IN: now reaches R1.2
- net VCA_IN: now also J3.5 (Pin_5)
- net +3.3V renamed ATTACK_3
- net AUDIO_CV_OUT_1 renamed DECAY_1
- net DECAY_1: now also RV_DECAY1.1
- net BTN_LED_1: no longer names the net of R1.1
- net BTN_LED_1: now also J_VCA_IN1.T
- net MIDI_4R renamed GATE_DEFAULT
- net GATE_DEFAULT: now also J5.1 (Pin_1)
- net MIDI_5T renamed GATE
- net GATE: now also J8.1 (Pin_1), J5.2 (Pin_2)
- net PULSE_IN: no longer names the net of R2.2
- net PULSE_IN: now also Q1.2 (B)
- new net: J_VCA_OUT1.T, R6.2
- new net: D1.1 (K), Q2.1 (E)
- new net: D1.2 (A), Q1.1 (E)
- new net: C1.1, R4.1, R5.2
- new net: J_VCA_CV1.T, R5.1
- new net: Q1.3 (C), R3.2
- new net A1_D3_R3: J8.6 (Pin_6), RV_ATTACK1.1, RV_DECAY1.2, RV_DECAY1.3, RV_RELEASE1.2, RV_RELEASE1.3
- new net ENV_OUT: J8.4 (Pin_4), JP_DEFAULT_ENV_TO_VCA1.1 (A), J_ENV_OUT1.T, R2.1
- new net ENV_OUT_DEFAULT: J5.3 (Pin_3), J_ENV_OUT1.TN
- new net RELEASE_1: J8.3 (Pin_3), RV_RELEASE1.1
- new net SUSTAIN_1: J6.2 (Pin_2), RV_SUSTAIN1.1
- new net SUSTAIN_2: J6.4 (Pin_4), RV_SUSTAIN1.2
- new net SUSTAIN_3: J6.6 (Pin_6), RV_SUSTAIN1.3
- new net VCA_CV: J3.3 (Pin_3), R4.2
- new net VCA_CV_DEFAULT: J5.5 (Pin_5), JP_DEFAULT_ENV_TO_VCA1.2 (B), J_VCA_CV1.TN
- new net VCA_IN_DEFAULT: J5.4 (Pin_4), J_VCA_IN1.TN
- new net VCA_OUT: J3.1 (Pin_1), R6.1
- new net VCA_OUT_DEFAULT: J5.6 (Pin_6), J_VCA_OUT1.TN
- no-connect marks 17 -> 6
Other:
- removed sheet LEDs
- note added: "Optional LP network to avoid pops on very short attack times. If you don't want to use this, just short R5 and don't solder C1."
- note added: "R1 & R6 is Only for testing"
- note added: "The higher the a pot resistance for Attack, Decay and Release pots is, the longer maximum time it'll have. A sweet spot can be around 200k or 500k. The BOM contains an A1M pot for these because of availability in 25mm height."
- note added: "There's a similar resistor on the core board, R1 and R6 are here for testing purposes. Should be shorted."
- note removed: "R15 only for testing purposes"
- title: Brain UI -> ADSR + VCA UI
- moved on the sheet: H1, H2, H4, J_GATE1, RV_ATTACK1
