File: modules/07-brain/electronics/core/brain-core.kicad_pcb (KiCad board)
At the start: 2 copper layers, 60.5 x 110 mm, 104 parts, among them J1 Conn_02x03_Odd_Even, J10 Conn_01x02, J11 Conn_01x01, J13 Conn_01x03, J2 Conn_02x02_Odd_Even, J3 Conn_02x02_Odd_Even, J4 Conn_02x03_Odd_Even, J5 Conn_01x02, J6 Conn_02x05_Odd_Even, J7 Conn_02x05_Odd_Even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

Commit message: Changed board versioning to 'rev' on Brain
Other:
- board text added: "BRAIN REV 3"
- board text removed: "SM-07 BRAIN V1.2"
Changed lines of the file:
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@@
 		)
 	)
-	(gr_text "SM-07 \nBRAIN\nV1.2"
+	(gr_text "BRAIN\nREV 3"
 		(at 148.384 122.354 0)
 		(layer "B.SilkS")
@@
 			(justify left bottom mirror)
 		)
-		(render_cache "SM-07 \nBRAIN\nV1.2" 0
-			(polygon
-				(pts
-					(xy 148.237661 117.265498) (xy 148.237661 117.562739) (xy 148.086829 117.562739) (xy 148.086829 117.265498)
-				)
-			)
-			(polygon
-				(pts
-					(xy 148.091323 117.558245) (xy 148.091323 117.709077) (xy 147.647745 117.709077) (xy 147.647745 117.558245)
-				)
-			)
-			(polygon
-				(pts
-					(xy 147.647745 118.143667) (xy 148.091323 118.143667) (xy 148.091323 118.2945) (xy 147.647745 118.2945)
-				)
-			)
-			(polygon
-				(pts
-					(xy 148.086829 118.148161) (xy 148.086829 117.997329) (xy 148.237661 117.997329) (xy 148.237661 118.148161)
-				)
-			)
-			(polygon
-				(pts
-					(xy 147.652239 117.704583) (xy 147.652239 118.148161) (xy 147.501336 118.148161) (xy 147.501336 117.704583)
-				)
-			)
-			(polygon
-				(pts
-					(xy 148.091323 117.11909) (xy 148.091323 117.269992) (xy 147.647745 117.269992) (xy 147.647745 117.11909)
-				)
-			)
-			(polygon
-				(pts
-					(xy 147.652239 117.265498) (xy 147.652239 117.41633) (xy 147.501336 117.41633) (xy 147.501336 117.265498)
-				)
-			)
-			(polygon
-				(pts
-					(xy 147.214137 117.11909) (xy 147.214137 118.2945) (xy 147.063305 118.2945) (xy 147.063305 117.562739)
-					(xy 146.916897 117.562739) (xy 146.916897 117.411836) (xy 147.063305 117.411836) (xy 147.063305 117.11909)
-				)
-			)
-			(polygon
-				(pts
-					(xy 146.628715 117.562739) (xy 146.628715 118.2945) (xy 146.477812 118.2945) (xy 146.477812 117.11909)
-					(xy 146.628715 117.11909) (xy 146.628715 117.411836) (xy 146.775053 117.411836) (xy 146.775053 117.562739)
-				)
-			)
-			(polygon
-				(pts
-					(xy 146.921391 117.558245) (xy 146.921391 117.855415) (xy 146.770559 117.855415) (xy 146.770559 117.558245)
-				)
-			)
-			(polygon
-				(pts
-					(xy 145.600697 117.704583) (xy 146.044275 117.704583) (xy 146.044275 117.855415) (xy 145.600697 117.855415)
-				)
-			)
-			(polygon
-				(pts
-					(xy 145.167089 117.265498) (xy 145.167089 118.148161) (xy 145.016257 118.148161) (xy 145.016257 117.855415)
-					(xy 144.869849 117.855415) (xy 144.869849 117.704583) (xy 145.016257 117.704583) (xy 145.016257 117.265498)
-				)
-			)
-			(polygon
-				(pts
-					(xy 145.020751 118.143667) (xy 145.020751 118.2945) (xy 144.577172 118.2945) (xy 144.577172 118.143667)
-				)
-			)
-			(polygon
-				(pts
-					(xy 145.020751 117.11909) (xy 145.020751 117.269992) (xy 144.577172 117.269992) (xy 144.577172 117.11909)
-				)
-			)
-			(polygon
-				(pts
-					(xy 144.581667 117.265498) (xy 144.581667 117.411836) (xy 144.728005 117.411836) (xy 144.728005 117.562739)
-					(xy 144.581667 117.562739) (xy 144.581667 118.148161) (xy 144.430764 118.148161) (xy 144.430764 117.265498)
-				)
-			)
-			(polygon
-				(pts
-					(xy 144.874343 117.558245) (xy 144.874343 117.709077) (xy 144.723511 117.709077) (xy 144.723511 117.558245)
-				)
-			)
-			(polygon
-				(pts
-					(xy 143.997227 117.850921) (xy 143.997227 118.2945) (xy 143.846325 118.2945) (xy 143.846325 117.850921)
-				)
-			)
-			(polygon
-				(pts
-					(xy 143.850819 117.704583) (xy 143.850819 117.855415) (xy 143.699987 117.855415) (xy 143.699987 117.704583)
-				)
-			)
-			(polygon
-				(pts
-					(xy 143.704481 117.558245) (xy 143.704481 117.709077) (xy 143.553648 117.709077) (xy 143.553648 117.558245)
-				)
-			)
-			(polygon
-				(pts
-					(xy 143.558142 117.269992) (xy 143.558142 117.562739) (xy 143.40724 117.562739) (xy 143.40724 117.11909)
-					(xy 144.143565 117.11909) (xy 144.143565 117.269992)
-				)
-			)
+		(render_cache "BRAIN\nREV 3" 0
 			(polygon
 				(pts
@@
 			(polygon
 				(pts
-					(xy 147.940421 122.012161) (xy 147.940421 121.714921) (xy 148.091323 121.714921) (xy 148.091323 122.012161)
+					(xy 148.237661 120.98309) (xy 148.237661 122.1585) (xy 148.086829 122.1585) (xy 148.086829 121.719415)
+					(xy 147.798577 121.719415) (xy 147.798577 121.865823) (xy 147.647745 121.865823) (xy 147.647745 121.568583)
+					(xy 148.086829 121.568583) (xy 148.086829 121.133992) (xy 147.647745 121.133992) (xy 147.647745 120.98309)
 				)
 			)
 			(polygon
 				(pts
-					(xy 147.944915 122.007667) (xy 147.944915 122.1585) (xy 147.794083 122.1585) (xy 147.794083 122.007667)
+					(xy 147.652239 121.129498) (xy 147.652239 121.573077) (xy 147.501336 121.573077) (xy 147.501336 121.129498)
 				)
 			)
 			(polygon
 				(pts
-					(xy 148.237661 120.98309) (xy 148.237661 121.719415) (xy 148.086829 121.719415) (xy 148.086829 120.98309)
+					(xy 147.652239 121.861329) (xy 147.652239 122.1585) (xy 147.501336 122.1585) (xy 147.501336 121.861329)
 				)
 			)
 			(polygon
 				(pts
-					(xy 147.652239 120.98309) (xy 147.652239 121.719415) (xy 147.501336 121.719415) (xy 147.501336 120.98309)
+					(xy 147.214137 120.98309) (xy 147.214137 122.1585) (xy 146.477812 122.1585) (xy 146.477812 122.007667)
+					(xy 147.063305 122.007667) (xy 147.063305 121.573077) (xy 146.624221 121.573077) (xy 146.624221 121.422245)
+					(xy 147.063305 121.422245) (xy 147.063305 121.133992) (xy 146.477812 121.133992) (xy 146.477812 120.98309)
 				)
 			)
 			(polygon
 				(pts
-					(xy 147.798577 121.714921) (xy 147.798577 122.012161) (xy 147.647745 122.012161) (xy 147.647745 121.714921)
+					(xy 145.893373 122.012161) (xy 145.893373 121.714921) (xy 146.044275 121.714921) (xy 146.044275 122.012161)
 				)
 			)
 			(polygon
 				(pts
-					(xy 146.921391 121.28033) (xy 146.921391 122.007667) (xy 147.214137 122.007667) (xy 147.214137 122.1585)
-					(xy 146.477812 122.1585) (xy 146.477812 122.007667) (xy 146.770559 122.007667) (xy 146.770559 120.98309)
-					(xy 146.921391 120.98309) (xy 146.921391 121.129498) (xy 147.214137 121.129498) (xy 147.214137 121.28033)
+					(xy 145.897867 122.007667) (xy 145.897867 122.1585) (xy 145.747035 122.1585) (xy 145.747035 122.007667)
 				)
 			)
 			(polygon
 				(pts
-					(xy 145.897867 121.861329) (xy 145.897867 122.1585) (xy 145.747035 122.1585) (xy 145.747035 121.861329)
+					(xy 146.190613 120.98309) (xy 146.190613 121.719415) (xy 146.039781 121.719415) (xy 146.039781 120.98309)
 				)
 			)
 			(polygon
 				(pts
-					(xy 145.167089 121.861329) (xy 145.167089 122.1585) (xy 144.430764 122.1585) (xy 144.430764 122.007667)
-					(xy 145.016257 122.007667) (xy 145.016257 121.861329)
+					(xy 145.605191 120.98309) (xy 145.605191 121.719415) (xy 145.454288 121.719415) (xy 145.454288 120.98309)
 				)
 			)
 			(polygon
 				(pts
-					(xy 144.577172 121.133992) (xy 144.577172 120.98309) (xy 145.020751 120.98309) (xy 145.020751 121.133992)
+					(xy 145.751529 121.714921) (xy 145.751529 122.012161) (xy 145.600697 122.012161) (xy 145.600697 121.714921)
 				)
 			)
 			(polygon
 				(pts
-					(xy 144.581667 121.129498) (xy 144.581667 121.426739) (xy 144.430764 121.426739) (xy 144.430764 121.129498)
+					(xy 144.143565 121.129498) (xy 144.143565 121.28033) (xy 143.992733 121.28033) (xy 143.992733 121.129498)
 				)
 			)
 			(polygon
 				(pts
-					(xy 145.020751 121.714921) (xy 145.020751 121.865823) (xy 144.869849 121.865823) (xy 144.869849 121.714921)
+					(xy 143.997227 120.98309) (xy 143.997227 121.133992) (xy 143.553648 121.133992) (xy 143.553648 120.98309)
 				)
 			)
 			(polygon
 				(pts
-					(xy 145.167089 121.129498) (xy 145.167089 121.28033) (xy 145.016257 121.28033) (xy 145.016257 121.129498)
+					(xy 143.558142 121.129498) (xy 143.558142 121.426739) (xy 143.40724 121.426739) (xy 143.40724 121.129498)
 				)
 			)
 			(polygon
 				(pts
-					(xy 144.728005 121.422245) (xy 144.728005 121.573077) (xy 144.577172 121.573077) (xy 144.577172 121.422245)
+					(xy 143.850819 121.422245) (xy 143.850819 121.573077) (xy 143.553648 121.573077) (xy 143.553648 121.422245)
 				)
 			)
 			(polygon
 				(pts
-					(xy 144.874343 121.568583) (xy 144.874343 121.719415) (xy 144.723511 121.719415) (xy 144.723511 121.568583)
+					(xy 143.558142 121.568583) (xy 143.558142 122.012161) (xy 143.40724 122.012161) (xy 143.40724 121.568583)
 				)
 			)
+			(polygon
+				(pts
+					(xy 143.553648 122.007667) (xy 143.997227 122.007667) (xy 143.997227 122.1585) (xy 143.553648 122.1585)
+				)
+			)
+			(polygon
+				(pts
+					(xy 143.992733 122.012161) (xy 143.992733 121.861329) (xy 144.143565 121.861329) (xy 144.143565 122.012161)
+				)
+			)
