File: modules/07-brain/electronics/core/brain-core.kicad_sch (KiCad schematic)
At the start: 12 parts, among them J1 Conn_02x03_Odd_Even, J10 Conn_01x02, J2 Conn_02x02_Odd_Even, J3 Conn_02x02_Odd_Even, J7 Conn_02x05_Odd_Even, J8 Conn_02x03_Odd_Even, J9 Conn_01x02

Commit message: Verfied JLCPCB for Brain 1.0
Other:
- company: (none) -> Shmøergh
- title: (none) -> Brain
Changed lines of the file:
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@@
 	(generator_version "9.0")
 	(paper "User" 340 210)
+	(title_block
+		(title "Brain")
+		(date "2025-12-11")
+		(company "Shmøergh")
+	)
 	(text "Power"
 		(exclude_from_sim no)

Commit message: Added Brain BOM
Parts:
- J1, J8: Mouser Part no. (none) -> 200-TSW10307TD; Part URL (none) -> https://mou.sr/4liCQlU
- J10, J9, J_DEV1: Mouser Part no. (none) -> 200-HTSW10207TS; Part URL (none) -> https://mou.sr/3IruU3e
- J2, J3: Mouser Part no. (none) -> 200-HTSW10207TD; Part URL (none) -> https://mou.sr/3TDBcz9
- J7: Mouser Part no. (none) -> 200-TSW10507TD; Part URL (none) -> https://mou.sr/40QhDaC
Changed lines of the file:
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@@
 			)
 		)
-		(property "Part URL" ""
+		(property "Part URL" "https://mou.sr/3TDBcz9"
 			(at 280.67 45.72 0)
 			(effects
@@
 		)
 		(property "Sim.Pins" ""
+			(at 280.67 45.72 0)
+			(effects
+				(font
+					(size 1.27 1.27)
+				)
+				(hide yes)
+			)
+		)
+		(property "Mouser Part no." "200-HTSW10207TD"
 			(at 280.67 45.72 0)
 			(effects
@@
 			)
 		)
-		(property "Part URL" ""
+		(property "Part URL" "https://mou.sr/40QhDaC"
 			(at 280.67 97.79 0)
 			(effects
@@
 		)
 		(property "Sim.Pins" ""
+			(at 280.67 97.79 0)
+			(effects
+				(font
+					(size 1.27 1.27)
+				)
+				(hide yes)
+			)
+		)
+		(property "Mouser Part no." "200-TSW10507TD"
 			(at 280.67 97.79 0)
 			(effects
@@
 			)
 		)
-		(property "Part URL" ""
+		(property "Part URL" "https://mou.sr/4liCQlU"
 			(at 280.67 143.51 0)
 			(effects
@@
 		)
 		(property "Sim.Pins" ""
+			(at 280.67 143.51 0)
+			(effects
+				(font
+					(size 1.27 1.27)
+				)
+				(hide yes)
+			)
+		)
+		(property "Mouser Part no." "200-TSW10307TD"
 			(at 280.67 143.51 0)
 			(effects
@@
 			)
 		)
-		(property "Part URL" ""
+		(property "Part URL" "https://mou.sr/3IruU3e"
 			(at 308.61 115.57 0)
 			(effects
@@
 		)
 		(property "Sim.Pins" ""
+			(at 308.61 115.57 0)
+			(effects
+				(font
+					(size 1.27 1.27)
+				)
+				(hide yes)
+			)
+		)
+		(property "Mouser Part no." "200-HTSW10207TS"
 			(at 308.61 115.57 0)
 			(effects
@@
 			)
 		)
-		(property "Part URL" ""
+		(property "Part URL" "https://mou.sr/3IruU3e"
 			(at 295.91 123.19 0)
 			(effects
@@
 		)
 		(property "Sim.Pins" ""
+			(at 295.91 123.19 0)
+			(effects
+				(font
+					(size 1.27 1.27)
+				)
+				(hide yes)
+			)
+		)
+		(property "Mouser Part no." "200-HTSW10207TS"
 			(at 295.91 123.19 0)
 			(effects
@@
 			)
 		)
-		(property "Part URL" ""
+		(property "Part URL" "https://mou.sr/3IruU3e"
 			(at 156.21 139.7 0)
 			(effects
@@
 		)
 		(property "LCSC" ""
+			(at 156.21 139.7 0)
+			(effects
+				(font
+					(size 1.27 1.27)
+				)
+				(hide yes)
+			)
+		)
+		(property "Mouser Part no." "200-HTSW10207TS"
 			(at 156.21 139.7 0)
 			(effects
@@
 			)
 		)
-		(property "Part URL" ""
+		(property "Part URL" "https://mou.sr/4liCQlU"
 			(at 280.67 62.23 0)
 			(effects
@@
 		)
 		(property "Sim.Pins" ""
+			(at 280.67 62.23 0)
+			(effects
+				(font
+					(size 1.27 1.27)
+				)
+				(hide yes)
+			)
+		)
+		(property "Mouser Part no." "200-TSW10307TD"
 			(at 280.67 62.23 0)
 			(effects
@@
 			)
 		)
-		(property "Part URL" ""
+		(property "Part URL" "https://mou.sr/3TDBcz9"
 			(at 280.67 77.47 0)
 			(effects
@@
 			(at 280.67 77.47 0)
 			(effects
+				(font
+					(size 1.27 1.27)
+				)
+				(hide yes)
+			)
+		)
+		(property "Mouser Part no." "200-HTSW10207TD"
+			(at 280.67 77.47 0)
+			(effects

Commit message: Changed Brain J_DEV header to horizontal
Parts:
- J_DEV1: footprint Connector_PinHeader_2.54mm:PinHeader_1x02_P2.54mm_Vertical -> Connector_PinHeader_2.54mm:PinHeader_1x02_P2.54mm_Horizontal; Mouser Part no. 200-HTSW10207TS -> 200-HTSW11008FSRA; Part URL https://mou.sr/3IruU3e -> https://mou.sr/4avMlMe
Connections:
- net MCU/UART_RX: now also J_DEV1.1 (Pin_1); no longer J_DEV1.2 (Pin_2)
- net MCU/UART_TX: now also J_DEV1.2 (Pin_2); no longer J_DEV1.1 (Pin_1)
Changed lines of the file:
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@@
 	(symbol
 		(lib_id "Connector_Generic:Conn_01x02")
-		(at 156.21 139.7 0)
+		(at 156.21 142.24 0)
+		(mirror x)
 		(unit 1)
 		(exclude_from_sim no)
@@
 		(on_board yes)
 		(dnp no)
-		(fields_autoplaced yes)
 		(property "Reference" "J_DEV1"
-			(at 158.75 139.6999 0)
+			(at 158.75 142.2401 0)
 			(effects
 				(font
@@
 		)
 		(property "Value" "Conn_01x02"
-			(at 158.75 142.2399 0)
+			(at 158.75 139.7001 0)
 			(effects
 				(font
@@
 			)
 		)
-		(property "Footprint" "Connector_PinHeader_2.54mm:PinHeader_1x02_P2.54mm_Vertical"
-			(at 156.21 139.7 0)
+		(property "Footprint" "Connector_PinHeader_2.54mm:PinHeader_1x02_P2.54mm_Horizontal"
+			(at 156.21 142.24 0)
 			(effects
 				(font
@@
 		)
 		(property "Datasheet" "~"
-			(at 156.21 139.7 0)
+			(at 156.21 142.24 0)
 			(effects
 				(font
@@
 		)
 		(property "Description" "Generic connector, single row, 01x02, script generated (kicad-library-utils/schlib/autogen/connector/)"
-			(at 156.21 139.7 0)
+			(at 156.21 142.24 0)
 			(effects
 				(font
@@
 		)
 		(property "Part No." ""
-			(at 156.21 139.7 0)
+			(at 156.21 142.24 0)
 			(effects
 				(font
@@
 			)
 		)
-		(property "Part URL" "https://mou.sr/3IruU3e"
-			(at 156.21 139.7 0)
+		(property "Part URL" "https://mou.sr/4avMlMe"
+			(at 156.21 142.24 0)
 			(effects
 				(font
@@
 		)
 		(property "Vendor" ""
-			(at 156.21 139.7 0)
+			(at 156.21 142.24 0)
 			(effects
 				(font
@@
 		)
 		(property "LCSC" ""
-			(at 156.21 139.7 0)
+			(at 156.21 142.24 0)
 			(effects
 				(font
@@
 			)
 		)
-		(property "Mouser Part no." "200-HTSW10207TS"
-			(at 156.21 139.7 0)
+		(property "Mouser Part no." "200-HTSW11008FSRA "
+			(at 156.21 142.24 0)
 			(effects
 				(font

Commit message: KiCAD version update - Brain
Other:
- title: Brain -> Brain Core
Changed lines of the file:
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@@
 	(paper "User" 340 210)
 	(title_block
-		(title "Brain")
-		(date "2025-12-11")
+		(title "Brain Core")
+		(date "2026-02-21")
+		(rev "v1.1")
 		(company "Shmøergh")
 	)
