File: modules/02-vco/electronics/core/sheets/sub+noise.kicad_sch (KiCad schematic)
At the start: 20 parts, among them Q6 BC847, Q7 MMBT5551, U8 TL072, U9 CD4040BM96

Commit message: KiCAD version updates - PSU + VCO
Other:
- company: (none) -> Shmøergh
- title: (none) -> Moduleur VCO core
Changed lines of the file:
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@@
 	(generator_version "9.0")
 	(paper "A4")
+	(title_block
+		(title "Moduleur VCO core")
+		(date "2026-02-21")
+		(rev "v1.0")
+		(company "Shmøergh")
+	)
 	(rectangle
 		(start 20.32 20.32)
