File: modules/02-vco/electronics/ui/vco-ui.kicad_sch (KiCad schematic)
At the start: 32 parts, among them J1 Conn_01x04, J2 Conn_02x05_Odd_Even, J3 Conn_02x03_Odd_Even, J4 Conn_01x02, J5 Conn_02x02_Counter_Clockwise, J6 Conn_01x07, U1 0203

Commit message: VCO JLCPCB export done for v1.0
Other:
- title: Hog Moduleur VCO UI -> Moduleur VCO UI
Changed lines of the file:
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@@
 	(paper "A4")
 	(title_block
-		(title "Hog Moduleur VCO UI")
-		(date "2025-10-24")
-		(rev "v0.2")
+		(title "Moduleur VCO UI")
+		(date "2025-12-11")
+		(rev "v1.0")
 		(company "Shmøergh")
 	)

Commit message: Added full BOM to VCO
Parts:
- R1: Part URL (none) -> https://mou.sr/3XNtowV; Part no. (none) -> 603-MFR-25FBF52-130K
- R4, R5: Part URL (none) -> https://mou.sr/44Vd3Kk; Part no. (none) -> 603-MFR-25FBF52-510K
Changed lines of the file:
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@@
+			)
+		)
+		(property "Part URL" "https://mou.sr/3XNtowV"
+			(at 50.8 57.15 0)
+			(effects
+				(font
+					(size 1.27 1.27)
+				)
+				(hide yes)
+			)
+		)
+		(property "Part no." "603-MFR-25FBF52-130K "
+			(at 50.8 57.15 0)
+			(effects
+				(font
+					(size 1.27 1.27)
+				)
+				(hide yes)
 			)
 		)
@@
 			)
 		)
+		(property "Part URL" "https://mou.sr/44Vd3Kk"
+			(at 109.22 77.47 0)
+			(effects
+				(font
+					(size 1.27 1.27)
+				)
+				(hide yes)
+			)
+		)
+		(property "Part no." "603-MFR-25FBF52-510K "
+			(at 109.22 77.47 0)
+			(effects
+				(font
+					(size 1.27 1.27)
+				)
+				(hide yes)
+			)
+		)
 		(pin "2"
 		)
@@
 			(at 109.22 57.15 0)
 			(effects
+				(font
+					(size 1.27 1.27)
+				)
+				(hide yes)
+			)
+		)
+		(property "Part URL" "https://mou.sr/44Vd3Kk"
+			(at 109.22 57.15 0)
+			(effects
+				(font
+					(size 1.27 1.27)
+				)
+				(hide yes)
+			)
+		)
+		(property "Part no." "603-MFR-25FBF52-510K "
+			(at 109.22 57.15 0)
+			(effects

Commit message: Fixed UI component part number bugs
Parts:
- RV_FINE1, RV_PWM1, RV_TUNE1: Part URL https://mou.sr/4694GMU -> https://mou.sr/41lYe2k; Part no. 652-PTV09A4025FB104 -> 652-PTV09A4025UB104
Changed lines of the file:
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@@
 			)
 		)
-		(property "Part URL" "https://mou.sr/4694GMU"
+		(property "Part URL" "https://mou.sr/41lYe2k"
 			(at 109.22 67.31 0)
 			(effects
@@
 			)
 		)
-		(property "Part no." "652-PTV09A4025FB104"
+		(property "Part no." "652-PTV09A4025UB104"
 			(at 109.22 67.31 0)
 			(effects
@@
 			)
 		)
-		(property "Part URL" "https://mou.sr/4694GMU"
+		(property "Part URL" "https://mou.sr/41lYe2k"
 			(at 165.1 67.31 0)
 			(effects
@@
 			)
 		)
-		(property "Part no." "652-PTV09A4025FB104"
+		(property "Part no." "652-PTV09A4025UB104"
 			(at 165.1 67.31 0)
 			(effects
@@
 			)
 		)
-		(property "Part URL" "https://mou.sr/4694GMU"
+		(property "Part URL" "https://mou.sr/41lYe2k"
 			(at 50.8 67.31 0)
 			(effects
@@
 			)
 		)
-		(property "Part no." "652-PTV09A4025FB104"
+		(property "Part no." "652-PTV09A4025UB104"
 			(at 50.8 67.31 0)
 			(effects

Commit message: Updated UI BOMs
Parts:
- RV_FINE1, RV_PWM1, RV_TUNE1: Note (none) -> Knurled Shaft
