File: modules/03-sidechain-mixer/electronics/core/sidechain-mixer-core.kicad_pcb (KiCad board)
At the start: 2 copper layers, 58 x 65 mm, 74 parts, among them J1 Conn_01x04, J2 Conn_02x05_Odd_Even, J3 Conn_02x05_Odd_Even, J4 Conn_01x02, J5 Conn_02x03_Odd_Even, J6 Conn_01x04, J8 Conn_01x06, Q1 BC847BS, U1 TL072, U2 TL072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

Commit message: Mixer JLCPCB verified for 1.0
Other:
- board text added: "SHMØERGH MODULEUR"
- board text added: "SM-03 Sidechain Mixer V1.0 / 2025 DEC"
- board text removed: "HM-03 Sidechain Mixer V0.1 / 2025 Aug"
- board text removed: "SHMØERGH HOG MODULEUR"

Commit message: KiCAD version update - Mixer + compressor
Other:
- board text added: "SM-03 Sidechain Mixer V1.0"
- board text removed: "SM-03 Sidechain Mixer V1.0 / 2025 DEC"

Commit message: Changed board versioning to 'rev' on VCO and Mixer
Other:
- board text added: "Sidechain Mixer REV 1"
- board text removed: "SM-03 Sidechain Mixer V1.0"
Changed lines of the file:
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@@
 		)
 	)
-	(gr_text "SM-03\nSidechain Mixer\nV1.0"
+	(gr_text "\nSidechain Mixer\nREV 1"
 		(at 136.065 126.931 0)
 		(layer "B.SilkS")
@@
 			(justify right bottom mirror)
 		)
-		(render_cache "SM-03\nSidechain Mixer\nV1.0" 0
-			(polygon
-				(pts
-					(xy 141.036281 121.842498) (xy 141.036281 122.139739) (xy 140.885449 122.139739) (xy 140.885449 121.842498)
-				)
-			)
-			(polygon
-				(pts
-					(xy 140.889943 122.135245) (xy 140.889943 122.286077) (xy 140.446365 122.286077) (xy 140.446365 122.135245)
-				)
-			)
-			(polygon
-				(pts
-					(xy 140.446365 122.720667) (xy 140.889943 122.720667) (xy 140.889943 122.8715) (xy 140.446365 122.8715)
-				)
-			)
-			(polygon
-				(pts
-					(xy 140.885449 122.725161) (xy 140.885449 122.574329) (xy 141.036281 122.574329) (xy 141.036281 122.725161)
-				)
-			)
-			(polygon
-				(pts
-					(xy 140.450859 122.281583) (xy 140.450859 122.725161) (xy 140.299956 122.725161) (xy 140.299956 122.281583)
-				)
-			)
-			(polygon
-				(pts
-					(xy 140.889943 121.69609) (xy 140.889943 121.846992) (xy 140.446365 121.846992) (xy 140.446365 121.69609)
-				)
-			)
-			(polygon
-				(pts
-					(xy 140.450859 121.842498) (xy 140.450859 121.99333) (xy 140.299956 121.99333) (xy 140.299956 121.842498)
-				)
-			)
-			(polygon
-				(pts
-					(xy 140.012757 121.69609) (xy 140.012757 122.8715) (xy 139.861925 122.8715) (xy 139.861925 122.139739)
-					(xy 139.715517 122.139739) (xy 139.715517 121.988836) (xy 139.861925 121.988836) (xy 139.861925 121.69609)
-				)
-			)
-			(polygon
-				(pts
-					(xy 139.427335 122.139739) (xy 139.427335 122.8715) (xy 139.276432 122.8715) (xy 139.276432 121.69609)
-					(xy 139.427335 121.69609) (xy 139.427335 121.988836) (xy 139.573673 121.988836) (xy 139.573673 122.139739)
-				)
-			)
-			(polygon
-				(pts
-					(xy 139.720011 122.135245) (xy 139.720011 122.432415) (xy 139.569179 122.432415) (xy 139.569179 122.135245)
-				)
-			)
-			(polygon
-				(pts
-					(xy 138.399317 122.281583) (xy 138.842895 122.281583) (xy 138.842895 122.432415) (xy 138.399317 122.432415)
-				)
-			)
-			(polygon
-				(pts
-					(xy 137.965709 121.842498) (xy 137.965709 122.725161) (xy 137.814877 122.725161) (xy 137.814877 122.432415)
-					(xy 137.668469 122.432415) (xy 137.668469 122.281583) (xy 137.814877 122.281583) (xy 137.814877 121.842498)
-				)
-			)
-			(polygon
-				(pts
-					(xy 137.819371 122.720667) (xy 137.819371 122.8715) (xy 137.375792 122.8715) (xy 137.375792 122.720667)
-				)
-			)
-			(polygon
-				(pts
-					(xy 137.819371 121.69609) (xy 137.819371 121.846992) (xy 137.375792 121.846992) (xy 137.375792 121.69609)
-				)
-			)
-			(polygon
-				(pts
-					(xy 137.380287 121.842498) (xy 137.380287 121.988836) (xy 137.526625 121.988836) (xy 137.526625 122.139739)
-					(xy 137.380287 122.139739) (xy 137.380287 122.725161) (xy 137.229384 122.725161) (xy 137.229384 121.842498)
-				)
-			)
-			(polygon
-				(pts
-					(xy 137.672963 122.135245) (xy 137.672963 122.286077) (xy 137.522131 122.286077) (xy 137.522131 122.135245)
-				)
-			)
-			(polygon
-				(pts
-					(xy 136.942185 121.842498) (xy 136.942185 121.99333) (xy 136.791353 121.99333) (xy 136.791353 121.842498)
-				)
-			)
-			(polygon
-				(pts
-					(xy 136.795847 121.69609) (xy 136.795847 121.846992) (xy 136.352268 121.846992) (xy 136.352268 121.69609)
-				)
-			)
-			(polygon
-				(pts
-					(xy 136.356762 121.842498) (xy 136.356762 122.139739) (xy 136.20586 122.139739) (xy 136.20586 121.842498)
-				)
-			)
-			(polygon
-				(pts
-					(xy 136.649439 122.135245) (xy 136.649439 122.286077) (xy 136.352268 122.286077) (xy 136.352268 122.135245)
-				)
-			)
-			(polygon
-				(pts
-					(xy 136.356762 122.281583) (xy 136.356762 122.725161) (xy 136.20586 122.725161) (xy 136.20586 122.281583)
-				)
-			)
-			(polygon
-				(pts
-					(xy 136.352268 122.720667) (xy 136.795847 122.720667) (xy 136.795847 122.8715) (xy 136.352268 122.8715)
-				)
-			)
-			(polygon
-				(pts
-					(xy 136.791353 122.725161) (xy 136.791353 122.574329) (xy 136.942185 122.574329) (xy 136.942185 122.725161)
-				)
-			)
+		(render_cache "\nSidechain Mixer\nREV 1" 0
 			(polygon
 				(pts
@@
 			(polygon
 				(pts
-					(xy 139.715517 126.589161) (xy 139.715517 126.291921) (xy 139.866419 126.291921) (xy 139.866419 126.589161)
-				)
-			)
-			(polygon
-				(pts
-					(xy 139.720011 126.584667) (xy 139.720011 126.7355) (xy 139.569179 126.7355) (xy 139.569179 126.584667)
-				)
-			)
-			(polygon
-				(pts
-					(xy 140.012757 125.56009) (xy 140.012757 126.296415) (xy 139.861925 126.296415) (xy 139.861925 125.56009)
-				)
-			)
-			(polygon
-				(pts
-					(xy 139.427335 125.56009) (xy 139.427335 126.296415) (xy 139.276432 126.296415) (xy 139.276432 125.56009)
-				)
-			)
-			(polygon
-				(pts
-					(xy 139.573673 126.291921) (xy 139.573673 126.589161) (xy 139.422841 126.589161) (xy 139.422841 126.291921)
-				)
-			)
-			(polygon
-				(pts
-					(xy 138.696487 125.85733) (xy 138.696487 126.584667) (xy 138.989233 126.584667) (xy 138.989233 126.7355)
-					(xy 138.252908 126.7355) (xy 138.252908 126.584667) (xy 138.545655 126.584667) (xy 138.545655 125.56009)
-					(xy 138.696487 125.56009) (xy 138.696487 125.706498) (xy 138.989233 125.706498) (xy 138.989233 125.85733)
-				)
-			)
-			(polygon
-				(pts
-					(xy 137.672963 126.438329) (xy 137.672963 126.7355) (xy 137.522131 126.7355) (xy 137.522131 126.438329)
-				)
-			)
-			(polygon
-				(pts
-					(xy 136.942185 125.706498) (xy 136.942185 126.589161) (xy 136.791353 126.589161) (xy 136.791353 126.296415)
-					(xy 136.644945 126.296415) (xy 136.644945 126.145583) (xy 136.791353 126.145583) (xy 136.791353 125.706498)
-				)
-			)
-			(polygon
-				(pts
-					(xy 136.795847 126.584667) (xy 136.795847 126.7355) (xy 136.352268 126.7355) (xy 136.352268 126.584667)
-				)
-			)
-			(polygon
-				(pts
-					(xy 136.795847 125.56009) (xy 136.795847 125.710992) (xy 136.352268 125.710992) (xy 136.352268 125.56009)
-				)
-			)
-			(polygon
-				(pts
-					(xy 136.356763 125.706498) (xy 136.356763 125.852836) (xy 136.503101 125.852836) (xy 136.503101 126.003739)
-					(xy 136.356763 126.003739) (xy 136.356763 126.589161) (xy 136.20586 126.589161) (xy 136.20586 125.706498)
-				)
-			)
-			(polygon
-				(pts
-					(xy 136.649439 125.999245) (xy 136.649439 126.150077) (xy 136.498607 126.150077) (xy 136.498607 125.999245)
-				)
-			)
+					(xy 141.036281 125.56009) (xy 141.036281 126.7355) (xy 140.885449 126.7355) (xy 140.885449 126.296415)
+					(xy 140.597197 126.296415) (xy 140.597197 126.442823) (xy 140.446365 126.442823) (xy 140.446365 126.145583)
+					(xy 140.885449 126.145583) (xy 140.885449 125.710992) (xy 140.446365 125.710992) (xy 140.446365 125.56009)
+				)
+			)
+			(polygon
+				(pts
+					(xy 140.450859 125.706498) (xy 140.450859 126.150077) (xy 140.299956 126.150077) (xy 140.299956 125.706498)
+				)
+			)
+			(polygon
+				(pts
+					(xy 140.450859 126.438329) (xy 140.450859 126.7355) (xy 140.299956 126.7355) (xy 140.299956 126.438329)
+				)
+			)
+			(polygon
+				(pts
+					(xy 140.012757 125.56009) (xy 140.012757 126.7355) (xy 139.276432 126.7355) (xy 139.276432 126.584667)
+					(xy 139.861925 126.584667) (xy 139.861925 126.150077) (xy 139.422841 126.150077) (xy 139.422841 125.999245)
+					(xy 139.861925 125.999245) (xy 139.861925 125.710992) (xy 139.276432 125.710992) (xy 139.276432 125.56009)
+				)
+			)
+			(polygon
+				(pts
+					(xy 138.691993 126.589161) (xy 138.691993 126.291921) (xy 138.842895 126.291921) (xy 138.842895 126.589161)
+				)
+			)
+			(polygon
+				(pts
+					(xy 138.696487 126.584667) (xy 138.696487 126.7355) (xy 138.545655 126.7355) (xy 138.545655 126.584667)
+				)
+			)
+			(polygon
+				(pts
+					(xy 138.989233 125.56009) (xy 138.989233 126.296415) (xy 138.838401 126.296415) (xy 138.838401 125.56009)
+				)
+			)
+			(polygon
+				(pts
+					(xy 138.403811 125.56009) (xy 138.403811 126.296415) (xy 138.252908 126.296415) (xy 138.252908 125.56009)
+				)
+			)
+			(polygon
+				(pts
+					(xy 138.550149 126.291921) (xy 138.550149 126.589161) (xy 138.399317 126.589161) (xy 138.399317 126.291921)
+				)
+			)
+			(polygon
+				(pts
+					(xy 136.649439 125.85733) (xy 136.649439 126.584667) (xy 136.942185 126.584667) (xy 136.942185 126.7355)
+					(xy 136.20586 126.7355) (xy 136.20586 126.584667) (xy 136.498607 126.584667) (xy 136.498607 125.56009)
+					(xy 136.649439 125.56009) (xy 136.649439 125.706498) (xy 136.942185 125.706498) (xy 136.942185 125.85733)
+				)
+			)

Commit message: Fixed Mixer Core schemo and PCB after fckckin KiCAD update
Parts:
- Q1: footprint Package_TO_SOT_SMD:SOT-363_SC-70-6 -> Shmoergh_Custom_Footprints:SOT-363_SC-70-6
Other:
- board text added: "Sidechain Mixer REV 2"
- board text removed: "Sidechain Mixer REV 1"
