File: modules/03-sidechain-mixer/electronics/core/sheets/power.kicad_sch (KiCad schematic)
At the start: 7 parts, among them J3 Conn_02x05_Odd_Even, J4 Conn_01x02, J5 Conn_02x03_Odd_Even

Commit message: Added full BOM to Mixer module
Parts:
- J3: CHECKED (none) -> YES; Mouser Part no. (none) -> 571-5103310-1; Part URL (none) -> https://mou.sr/3GwYxj9
- J4: CHECKED (none) -> YES; Mouser Part no. (none) -> 200-HTSW10207TS; Part URL (none) -> https://mou.sr/3IruU3e
- J5: CHECKED (none) -> YES; Mouser Part no. (none) -> 200-TSW10307TD; Part URL (none) -> https://mou.sr/4liCQlU
Changed lines of the file:
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@@
 			)
 		)
-		(property "Part URL" ""
+		(property "Part URL" "https://mou.sr/4liCQlU"
 			(at 88.9 92.71 0)
 			(effects
@@
 			)
 		)
-		(property "CHECKED" ""
+		(property "CHECKED" "YES"
 			(at 88.9 92.71 0)
 			(effects
@@
 			)
 		)
-		(property "Mouser Part no." ""
+		(property "Mouser Part no." "200-TSW10307TD"
 			(at 88.9 92.71 0)
 			(effects
@@
 			)
 		)
-		(property "Part URL" ""
+		(property "Part URL" "https://mou.sr/3GwYxj9"
 			(at 156.21 97.79 0)
 			(effects
@@
 			)
 		)
-		(property "CHECKED" ""
+		(property "CHECKED" "YES"
 			(at 156.21 97.79 0)
 			(effects
@@
 			)
 		)
-		(property "Mouser Part no." ""
+		(property "Mouser Part no." "571-5103310-1"
 			(at 156.21 97.79 0)
 			(effects
@@
 			)
 		)
-		(property "Part URL" ""
+		(property "Part URL" "https://mou.sr/3IruU3e"
 			(at 92.71 109.22 0)
 			(effects
@@
 			)
 		)
-		(property "CHECKED" ""
+		(property "CHECKED" "YES"
 			(at 92.71 109.22 0)
 			(effects
@@
 			)
 		)
-		(property "Mouser Part no." ""
+		(property "Mouser Part no." "200-HTSW10207TS"
 			(at 92.71 109.22 0)
 			(effects

Commit message: Updated out-of-stock 100uF cap JLCPCB product no's
Parts:
- C23, C24: LCSC C2836437 -> C2836442
Changed lines of the file:
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@@
 			)
 		)
-		(property "LCSC" "C2836437"
+		(property "LCSC" "C2836442"
 			(at 231.14 91.44 0)
 			(effects
@@
 			)
 		)
-		(property "LCSC" "C2836437"
+		(property "LCSC" "C2836442"
 			(at 231.14 99.06 0)
 			(effects

Commit message: KiCAD version updates - PSU + VCO
Other:
- company: (none) -> Shmøergh
- title: (none) -> Moduleur Mixer & sidechain compressor
Changed lines of the file:
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@@
 	(generator_version "9.0")
 	(paper "A4")
+	(title_block
+		(title "Moduleur Mixer & sidechain compressor")
+		(date "2025-12-11")
+		(rev "v1.0")
+		(company "Shmøergh")
+	)
 	(text "UI power connection"
 		(exclude_from_sim no)
