File: modules/03-sidechain-mixer/electronics/core/sheets/sc-mixer.kicad_sch (KiCad schematic)
At the start: 57 parts, among them Q1 BC847BS, U1 TL072, U2 TL072, U3 TL072, U4 TL072

Commit message: Mixer JLCPCB verified for 1.0
Parts:
- R18, R19, R26, R28, R29, RV_ATTACK1, RV_BIAS1, RV_COMP1, RV_RELEASE1: Vendor (none) -> Mouser
Changed lines of the file:
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@@
 			)
 		)
+		(property "Vendor" "Mouser"
+			(at 144.78 74.93 0)
+			(effects
+				(font
+					(size 1.27 1.27)
+				)
+				(hide yes)
+			)
+		)
 		(pin "2"
 		)
@@
 			)
 		)
-		(property "Vendor" ""
+		(property "Vendor" "Mouser"
 			(at 146.05 118.11 90)
 			(effects
@@
 			)
 		)
-		(property "Vendor" ""
+		(property "Vendor" "Mouser"
 			(at 128.27 134.62 90)
 			(effects
@@
 			)
 		)
-		(property "Vendor" ""
+		(property "Vendor" "Mouser"
 			(at 135.89 139.7 90)
 			(effects
@@
 			)
 		)
-		(property "Vendor" ""
+		(property "Vendor" "Mouser"
 			(at 34.29 193.04 90)
 			(effects
@@
 			)
 		)
-		(property "Vendor" ""
+		(property "Vendor" "Mouser"
 			(at 88.9 137.16 0)
 			(effects
@@
 			)
 		)
+		(property "Vendor" "Mouser"
+			(at 207.01 26.67 90)
+			(effects
+				(font
+					(size 1.27 1.27)
+				)
+				(hide yes)
+			)
+		)
 		(pin "2"
 		)
@@
 			)
 		)
-		(property "Vendor" ""
+		(property "Vendor" "Mouser"
 			(at 58.42 129.54 0)
 			(effects
@@
 			)
 		)
-		(property "Vendor" ""
+		(property "Vendor" "Mouser"
 			(at 128.27 129.54 90)
 			(effects

Commit message: Added full BOM to Mixer module
Parts:
- R18, R19, R26, R28, R29: CHECKED (none) -> YES; Mouser Part no. (none) -> 603-MFR-25FRF5210K; Part URL (none) -> https://mou.sr/4aLzHIM
- RV_ATTACK1, RV_COMP1, RV_RELEASE1: CHECKED (none) -> YES; Mouser Part no. (none) -> 774-06TR4AA103CP; Part URL (none) -> https://mou.sr/44pTlq5
- RV_BIAS1: CHECKED (none) -> YES; Mouser Part no. (none) -> 774-06TR4AA104CP; Part URL (none) -> https://mou.sr/4oMQfnb
Changed lines of the file:
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@@
 			)
 		)
+		(property "CHECKED" "YES"
+			(at 144.78 74.93 0)
+			(effects
+				(font
+					(size 1.27 1.27)
+				)
+				(hide yes)
+			)
+		)
+		(property "Mouser Part no." "774-06TR4AA104CP"
+			(at 144.78 74.93 0)
+			(effects
+				(font
+					(size 1.27 1.27)
+				)
+				(hide yes)
+			)
+		)
+		(property "Part URL" "https://mou.sr/4oMQfnb"
+			(at 144.78 74.93 0)
+			(effects
+				(font
+					(size 1.27 1.27)
+				)
+				(hide yes)
+			)
+		)
 		(pin "2"
 		)
@@
 			)
 		)
-		(property "CHECKED" ""
+		(property "CHECKED" "YES"
 			(at 146.05 118.11 90)
 			(effects
@@
 			)
 		)
-		(property "Part URL" ""
+		(property "Part URL" "https://mou.sr/4aLzHIM"
 			(at 146.05 118.11 0)
 			(effects
@@
 			)
 		)
+		(property "Mouser Part no." "603-MFR-25FRF5210K"
+			(at 146.05 118.11 90)
+			(effects
+				(font
+					(size 1.27 1.27)
+				)
+				(hide yes)
+			)
+		)
 		(pin "1"
 		)
@@
 			)
 		)
-		(property "CHECKED" ""
+		(property "CHECKED" "YES"
 			(at 128.27 134.62 90)
 			(effects
@@
 			)
 		)
-		(property "Part URL" ""
+		(property "Part URL" "https://mou.sr/4aLzHIM"
 			(at 128.27 134.62 0)
 			(effects
@@
 			)
 		)
+		(property "Mouser Part no." "603-MFR-25FRF5210K"
+			(at 128.27 134.62 90)
+			(effects
+				(font
+					(size 1.27 1.27)
+				)
+				(hide yes)
+			)
+		)
 		(pin "1"
 		)
@@
 			)
 		)
-		(property "CHECKED" ""
+		(property "CHECKED" "YES"
 			(at 135.89 139.7 90)
 			(effects
@@
 			)
 		)
-		(property "Part URL" ""
+		(property "Part URL" "https://mou.sr/4aLzHIM"
 			(at 135.89 139.7 0)
 			(effects
@@
 			)
 		)
+		(property "Mouser Part no." "603-MFR-25FRF5210K"
+			(at 135.89 139.7 0)
+			(effects
+				(font
+					(size 1.27 1.27)
+				)
+				(hide yes)
+			)
+		)
 		(pin "1"
 		)
@@
 			)
 		)
-		(property "CHECKED" ""
+		(property "CHECKED" "YES"
 			(at 34.29 193.04 90)
 			(effects
@@
 			)
 		)
-		(property "Part URL" ""
+		(property "Part URL" "https://mou.sr/4aLzHIM"
 			(at 34.29 193.04 0)
 			(effects
@@
 			)
 		)
+		(property "Mouser Part no." "603-MFR-25FRF5210K"
+			(at 34.29 193.04 0)
+			(effects
+				(font
+					(size 1.27 1.27)
+				)
+				(hide yes)
+			)
+		)
 		(pin "1"
 		)
@@
 			)
 		)
-		(property "Part URL" ""
+		(property "Part URL" "https://mou.sr/44pTlq5"
 			(at 88.9 137.16 0)
 			(effects
@@
 			)
 		)
+		(property "CHECKED" "YES"
+			(at 88.9 137.16 0)
+			(effects
+				(font
+					(size 1.27 1.27)
+				)
+				(hide yes)
+			)
+		)
+		(property "Mouser Part no." "774-06TR4AA103CP"
+			(at 88.9 137.16 0)
+			(effects
+				(font
+					(size 1.27 1.27)
+				)
+				(hide yes)
+			)
+		)
 		(pin "2"
 		)
@@
 			)
 		)
+		(property "CHECKED" "YES"
+			(at 207.01 26.67 90)
+			(effects
+				(font
+					(size 1.27 1.27)
+				)
+				(hide yes)
+			)
+		)
+		(property "Mouser Part no." "774-06TR4AA103CP"
+			(at 207.01 26.67 90)
+			(effects
+				(font
+					(size 1.27 1.27)
+				)
+				(hide yes)
+			)
+		)
+		(property "Part URL" "https://mou.sr/44pTlq5"
+			(at 207.01 26.67 90)
+			(effects
+				(font
+					(size 1.27 1.27)
+				)
+				(hide yes)
+			)
+		)
 		(pin "2"
 		)
@@
 			)
 		)
-		(property "Part URL" ""
+		(property "Part URL" "https://mou.sr/44pTlq5"
 			(at 58.42 129.54 0)
 			(effects
@@
 			)
 		)
+		(property "CHECKED" "YES"
+			(at 58.42 129.54 90)
+			(effects
+				(font
+					(size 1.27 1.27)
+				)
+				(hide yes)
+			)
+		)
+		(property "Mouser Part no." "774-06TR4AA103CP"
+			(at 58.42 129.54 90)
+			(effects
+				(font
+					(size 1.27 1.27)
+				)
+				(hide yes)
+			)
+		)
 		(pin "2"
 		)
@@
 			)
 		)
-		(property "CHECKED" ""
+		(property "CHECKED" "YES"
 			(at 128.27 129.54 90)
 			(effects
@@
 			)
 		)
-		(property "Part URL" ""
+		(property "Part URL" "https://mou.sr/4aLzHIM"
 			(at 128.27 129.54 0)
 			(effects
@@
 			(at 128.27 129.54 90)
 			(effects
+				(font
+					(size 1.27 1.27)
+				)
+				(hide yes)
+			)
+		)
+		(property "Mouser Part no." "603-MFR-25FRF5210K"
+			(at 128.27 129.54 90)
+			(effects

Commit message: KiCAD version updates - PSU + VCO
Other:
- company: (none) -> Shmøergh
- title: (none) -> Moduleur Mixer & sidechain compressor
Changed lines of the file:
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@@
 	(generator_version "9.0")
 	(paper "User" 350 230)
+	(title_block
+		(title "Moduleur Mixer & sidechain compressor")
+		(date "2025-12-11")
+		(rev "v1.0")
+		(company "Shmøergh")
+	)
 	(rectangle
 		(start 269.24 15.24)

Commit message: Fixed Mixer Core schemo and PCB after fckckin KiCAD update
Parts:
- Q1: footprint Package_TO_SOT_SMD:SOT-363_SC-70-6 -> Shmoergh_Custom_Footprints:SOT-363_SC-70-6
