File: modules/03-sidechain-mixer/electronics/ui/sidechain-mixer-ui.kicad_pcb (KiCad board)
At the start: 2 copper layers, 58 x 110 mm, 36 parts, among them J1 Conn_02x03_Odd_Even, J2 Conn_02x05_Odd_Even, J3 Conn_01x04, J4 Conn_01x02, J5 Conn_01x06, J7 Conn_01x04

Commit message: Mixer JLCPCB verified for 1.0
Other:
- board text added: "SHMØERGH MODULEUR"
- board text added: "SM-03 SIDECHAIN MIXER UI V1.0 2025 DEC"
- board text removed: "HM-03 SIDECHAIN MIXER UI V0.2 2025 AUG"
- board text removed: "SHMØERGH HOG MODULEUR"

Commit message: Fixed socket to header on mixer UI
Parts:
- J3, J7: footprint Connector_PinHeader_2.54mm:PinHeader_1x04_P2.54mm_Vertical -> Connector_PinSocket_2.54mm:PinSocket_1x04_P2.54mm_Vertical

Commit message: KiCAD version update - Mixer + compressor
Other:
- board text added: "SM-03 SIDECHAIN MIXER UI V1.0"
- board text removed: "SM-03 SIDECHAIN MIXER UI V1.0 2025 DEC"
Changed lines of the file:
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@@
 		)
 	)
-	(gr_text "SM-03 SIDECHAIN\nMIXER UI\nV1.0 2025 DEC"
+	(gr_text "SM-03 SIDECHAIN\nMIXER UI\nV1.0"
 		(at 172.895 50.858 0)
 		(layer "F.SilkS")
@@
 			(justify right bottom)
 		)
-		(render_cache "SM-03 SIDECHAIN\nMIXER UI\nV1.0 2025 DEC" 0
+		(render_cache "SM-03 SIDECHAIN\nMIXER UI\nV1.0" 0
 			(polygon
 				(pts
@@
 			(polygon
 				(pts
-					(xy 161.70654 50.560749) (xy 161.70654 50.306187) (xy 161.579229 50.306187) (xy 161.579229 50.560749)
-				)
-			)
-			(polygon
-				(pts
-					(xy 161.70654 50.560749) (xy 161.70654 50.688) (xy 161.833791 50.688) (xy 161.833791 50.560749)
-				)
-			)
-			(polygon
-				(pts
-					(xy 161.451978 49.669812) (xy 161.451978 50.306187) (xy 161.579229 50.306187) (xy 161.579229 49.669812)
-				)
-			)
-			(polygon
-				(pts
-					(xy 161.961041 49.669812) (xy 161.961041 50.306187) (xy 162.088353 50.306187) (xy 162.088353 49.669812)
-				)
-			)
-			(polygon
-				(pts
-					(xy 161.833791 50.306187) (xy 161.833791 50.560749) (xy 161.961041 50.560749) (xy 161.961041 50.306187)
-				)
-			)
-			(polygon
-				(pts
-					(xy 162.596561 49.924374) (xy 162.596561 50.560749) (xy 162.341999 50.560749) (xy 162.341999 50.688)
-					(xy 162.978374 50.688) (xy 162.978374 50.560749) (xy 162.723812 50.560749) (xy 162.723812 49.669812)
-					(xy 162.596561 49.669812) (xy 162.596561 49.797124) (xy 162.341999 49.797124) (xy 162.341999 49.924374)
-				)
-			)
-			(polygon
-				(pts
-					(xy 163.486582 50.433498) (xy 163.486582 50.688) (xy 163.613833 50.688) (xy 163.613833 50.433498)
-				)
-			)
-			(polygon
-				(pts
-					(xy 164.122041 49.797124) (xy 164.122041 50.560749) (xy 164.249291 50.560749) (xy 164.249291 50.306187)
-					(xy 164.376603 50.306187) (xy 164.376603 50.178936) (xy 164.249291 50.178936) (xy 164.249291 49.797124)
-				)
-			)
-			(polygon
-				(pts
-					(xy 164.249291 50.560749) (xy 164.249291 50.688) (xy 164.631104 50.688) (xy 164.631104 50.560749)
-				)
-			)
-			(polygon
-				(pts
-					(xy 164.249291 49.669812) (xy 164.249291 49.797124) (xy 164.631104 49.797124) (xy 164.631104 49.669812)
-				)
-			)
-			(polygon
-				(pts
-					(xy 164.631104 49.797124) (xy 164.631104 49.924374) (xy 164.503853 49.924374) (xy 164.503853 50.051686)
-					(xy 164.631104 50.051686) (xy 164.631104 50.560749) (xy 164.758416 50.560749) (xy 164.758416 49.797124)
-				)
-			)
-			(polygon
-				(pts
-					(xy 164.376603 50.051686) (xy 164.376603 50.178936) (xy 164.503853 50.178936) (xy 164.503853 50.051686)
-				)
-			)
-			(polygon
-				(pts
-					(xy 165.902083 50.433498) (xy 165.902083 50.688) (xy 166.538457 50.688) (xy 166.538457 50.560749)
-					(xy 166.029333 50.560749) (xy 166.029333 50.433498)
-				)
-			)
-			(polygon
-				(pts
-					(xy 166.411146 49.797124) (xy 166.411146 49.669812) (xy 166.029333 49.669812) (xy 166.029333 49.797124)
-				)
-			)
-			(polygon
-				(pts
-					(xy 166.411146 49.797124) (xy 166.411146 50.051686) (xy 166.538457 50.051686) (xy 166.538457 49.797124)
-				)
-			)
-			(polygon
-				(pts
-					(xy 166.029333 50.306187) (xy 166.029333 50.433498) (xy 166.156645 50.433498) (xy 166.156645 50.306187)
-				)
-			)
-			(polygon
-				(pts
-					(xy 165.902083 49.797124) (xy 165.902083 49.924374) (xy 166.029333 49.924374) (xy 166.029333 49.797124)
-				)
-			)
-			(polygon
-				(pts
-					(xy 166.283895 50.051686) (xy 166.283895 50.178936) (xy 166.411146 50.178936) (xy 166.411146 50.051686)
-				)
-			)
-			(polygon
-				(pts
-					(xy 166.156645 50.178936) (xy 166.156645 50.306187) (xy 166.283895 50.306187) (xy 166.283895 50.178936)
-				)
-			)
-			(polygon
-				(pts
-					(xy 166.792104 49.797124) (xy 166.792104 50.560749) (xy 166.919354 50.560749) (xy 166.919354 50.306187)
-					(xy 167.046666 50.306187) (xy 167.046666 50.178936) (xy 166.919354 50.178936) (xy 166.919354 49.797124)
-				)
-			)
-			(polygon
-				(pts
-					(xy 166.919354 50.560749) (xy 166.919354 50.688) (xy 167.301167 50.688) (xy 167.301167 50.560749)
-				)
-			)
-			(polygon
-				(pts
-					(xy 166.919354 49.669812) (xy 166.919354 49.797124) (xy 167.301167 49.797124) (xy 167.301167 49.669812)
-				)
-			)
-			(polygon
-				(pts
-					(xy 167.301167 49.797124) (xy 167.301167 49.924374) (xy 167.173916 49.924374) (xy 167.173916 50.051686)
-					(xy 167.301167 50.051686) (xy 167.301167 50.560749) (xy 167.428478 50.560749) (xy 167.428478 49.797124)
-				)
-			)
-			(polygon
-				(pts
-					(xy 167.046666 50.051686) (xy 167.046666 50.178936) (xy 167.173916 50.178936) (xy 167.173916 50.051686)
-				)
-			)
-			(polygon
-				(pts
-					(xy 167.682125 50.433498) (xy 167.682125 50.688) (xy 168.318499 50.688) (xy 168.318499 50.560749)
-					(xy 167.809375 50.560749) (xy 167.809375 50.433498)
-				)
-			)
-			(polygon
-				(pts
-					(xy 168.191188 49.797124) (xy 168.191188 49.669812) (xy 167.809375 49.669812) (xy 167.809375 49.797124)
-				)
-			)
-			(polygon
-				(pts
-					(xy 168.191188 49.797124) (xy 168.191188 50.051686) (xy 168.318499 50.051686) (xy 168.318499 49.797124)
-				)
-			)
-			(polygon
-				(pts
-					(xy 167.809375 50.306187) (xy 167.809375 50.433498) (xy 167.936687 50.433498) (xy 167.936687 50.306187)
-				)
-			)
-			(polygon
-				(pts
-					(xy 167.682125 49.797124) (xy 167.682125 49.924374) (xy 167.809375 49.924374) (xy 167.809375 49.797124)
-				)
-			)
-			(polygon
-				(pts
-					(xy 168.063937 50.051686) (xy 168.063937 50.178936) (xy 168.191188 50.178936) (xy 168.191188 50.051686)
-				)
-			)
-			(polygon
-				(pts
-					(xy 167.936687 50.178936) (xy 167.936687 50.306187) (xy 168.063937 50.306187) (xy 168.063937 50.178936)
-				)
-			)
-			(polygon
-				(pts
-					(xy 168.572146 49.669812) (xy 168.572146 50.178936) (xy 169.081209 50.178936) (xy 169.081209 50.051686)
-					(xy 168.699396 50.051686) (xy 168.699396 49.797124) (xy 169.20852 49.797124) (xy 169.20852 49.669812)
-				)
-			)
-			(polygon
-				(pts
-					(xy 169.081209 50.178936) (xy 169.081209 50.560749) (xy 169.20852 50.560749) (xy 169.20852 50.178936)
-				)
-			)
-			(polygon
-				(pts
-					(xy 169.081209 50.560749) (xy 168.699396 50.560749) (xy 168.699396 50.688) (xy 169.081209 50.688)
-				)
-			)
-			(polygon
-				(pts
-					(xy 168.699396 50.560749) (xy 168.699396 50.433498) (xy 168.572146 50.433498) (xy 168.572146 50.560749)
-				)
-			)
-			(polygon
-				(pts
-					(xy 170.352187 49.669812) (xy 170.352187 50.688) (xy 170.861251 50.688) (xy 170.861251 50.560749)
-					(xy 170.479438 50.560749) (xy 170.479438 49.797124) (xy 170.861251 49.797124) (xy 170.861251 49.669812)
-				)
-			)
-			(polygon
-				(pts
-					(xy 170.861251 49.797124) (xy 170.861251 50.560749) (xy 170.988562 50.560749) (xy 170.988562 49.797124)
-				)
-			)
-			(polygon
-				(pts
-					(xy 171.242208 49.669812) (xy 171.242208 50.688) (xy 171.878583 50.688) (xy 171.878583 50.560749)
-					(xy 171.369459 50.560749) (xy 171.369459 50.178936) (xy 171.751271 50.178936) (xy 171.751271 50.051686)
-					(xy 171.369459 50.051686) (xy 171.369459 49.797124) (xy 171.878583 49.797124) (xy 171.878583 49.669812)
-				)
-			)
-			(polygon
-				(pts
-					(xy 172.132229 49.797124) (xy 172.132229 50.560749) (xy 172.25948 50.560749) (xy 172.25948 49.797124)
-				)
-			)
-			(polygon
-				(pts
-					(xy 172.25948 50.560749) (xy 172.25948 50.688) (xy 172.641292 50.688) (xy 172.641292 50.560749)
-				)
-			)
-			(polygon
-				(pts
-					(xy 172.641292 50.433498) (xy 172.641292 50.560749) (xy 172.768604 50.560749) (xy 172.768604 50.433498)
-				)
-			)
-			(polygon
-				(pts
-					(xy 172.25948 49.669812) (xy 172.25948 49.797124) (xy 172.641292 49.797124) (xy 172.641292 49.669812)
-				)
-			)
-			(polygon
-				(pts
-					(xy 172.641292 49.797124) (xy 172.641292 49.924374) (xy 172.768604 49.924374) (xy 172.768604 49.797124)
-				)
-			)
+					(xy 169.716729 50.560749) (xy 169.716729 50.306187) (xy 169.589418 50.306187) (xy 169.589418 50.560749)
+				)
+			)
+			(polygon
+				(pts
+					(xy 169.716729 50.560749) (xy 169.716729 50.688) (xy 169.84398 50.688) (xy 169.84398 50.560749)
+				)
+			)
+			(polygon
+				(pts
+					(xy 169.462167 49.669812) (xy 169.462167 50.306187) (xy 169.589418 50.306187) (xy 169.589418 49.669812)
+				)
+			)
+			(polygon
+				(pts
+					(xy 169.97123 49.669812) (xy 169.97123 50.306187) (xy 170.098542 50.306187) (xy 170.098542 49.669812)
+				)
+			)
+			(polygon
+				(pts
+					(xy 169.84398 50.306187) (xy 169.84398 50.560749) (xy 169.97123 50.560749) (xy 169.97123 50.306187)
+				)
+			)
+			(polygon
+				(pts
+					(xy 170.60675 49.924374) (xy 170.60675 50.560749) (xy 170.352188 50.560749) (xy 170.352188 50.688)
+					(xy 170.988563 50.688) (xy 170.988563 50.560749) (xy 170.734001 50.560749) (xy 170.734001 49.669812)
+					(xy 170.60675 49.669812) (xy 170.60675 49.797124) (xy 170.352188 49.797124) (xy 170.352188 49.924374)
+				)
+			)
+			(polygon
+				(pts
+					(xy 171.496771 50.433498) (xy 171.496771 50.688) (xy 171.624022 50.688) (xy 171.624022 50.433498)
+				)
+			)
+			(polygon
+				(pts
+					(xy 172.13223 49.797124) (xy 172.13223 50.560749) (xy 172.25948 50.560749) (xy 172.25948 50.306187)
+					(xy 172.386792 50.306187) (xy 172.386792 50.178936) (xy 172.25948 50.178936) (xy 172.25948 49.797124)
+				)
+			)
+			(polygon
+				(pts
+					(xy 172.25948 50.560749) (xy 172.25948 50.688) (xy 172.641293 50.688) (xy 172.641293 50.560749)
+				)
+			)
+			(polygon
+				(pts
+					(xy 172.25948 49.669812) (xy 172.25948 49.797124) (xy 172.641293 49.797124) (xy 172.641293 49.669812)
+				)
+			)
+			(polygon
+				(pts
+					(xy 172.641293 49.797124) (xy 172.641293 49.924374) (xy 172.514042 49.924374) (xy 172.514042 50.051686)
+					(xy 172.641293 50.051686) (xy 172.641293 50.560749) (xy 172.768605 50.560749) (xy 172.768605 49.797124)
+				)
+			)
+			(polygon
+				(pts
+					(xy 172.386792 50.051686) (xy 172.386792 50.178936) (xy 172.514042 50.178936) (xy 172.514042 50.051686)
+				)
+			)

Commit message: Changed board versioning to 'rev' on VCO and Mixer
Other:
- board text added: "SIDECHAIN MIXER UI REV 1"
- board text removed: "SM-03 SIDECHAIN MIXER UI V1.0"

Commit message: Fixed Mixer UI schemo and PCB after fckckin KiCAD update
Other:
- board text added: "SIDECHAIN MIXER UI REV 2"
- board text removed: "SIDECHAIN MIXER UI REV 1"
