File: modules/03-sidechain-mixer/electronics/ui/sidechain-mixer-ui.kicad_sch (KiCad schematic)
At the start: 29 parts, among them J1 Conn_02x03_Odd_Even, J2 Conn_02x05_Odd_Even, J3 Conn_01x04, J4 Conn_01x02, J5 Conn_01x06, J7 Conn_01x04

Commit message: Added full BOM to Mixer module
Parts:
- J2: Part URL (none) -> https://mou.sr/4lVCZM9; Part no. (none) -> 200-SSW10501TD; Vendor (none) -> Mouser
- J3, J7: Part URL (none) -> https://mou.sr/4kxE3Vr; Part no. (none) -> 200-SSW10401TMS; Vendor (none) -> Mouser
- R1: Part URL (none) -> https://mou.sr/4aLzHIM; Part no. (none) -> 603-MFR-25FRF5210K; Vendor (none) -> Mouser
- R3: Part URL (none) -> https://mou.sr/3PSKVAZ; Part no. (none) -> 603-MFR-25FRF5220K; Vendor (none) -> Mouser
Changed lines of the file:
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@@
 			)
 		)
-		(property "Part URL" ""
+		(property "Part URL" "https://mou.sr/4kxE3Vr"
 			(at 139.7 148.59 0)
 			(effects
@@
 			)
 		)
-		(property "Vendor" ""
+		(property "Vendor" "Mouser"
 			(at 139.7 148.59 0)
 			(effects
@@
 			)
 		)
+		(property "Part no." "200-SSW10401TMS"
+			(at 139.7 148.59 0)
+			(effects
+				(font
+					(size 1.27 1.27)
+				)
+				(hide yes)
+			)
+		)
 		(pin "3"
 		)
@@
 			)
 		)
-		(property "Part URL" ""
+		(property "Part URL" "https://mou.sr/4lVCZM9"
 			(at 87.63 149.86 0)
 			(effects
@@
 			)
 		)
-		(property "Vendor" ""
+		(property "Vendor" "Mouser"
 			(at 87.63 149.86 0)
 			(effects
@@
 			)
 		)
+		(property "Part no." "200-SSW10501TD"
+			(at 87.63 149.86 0)
+			(effects
+				(font
+					(size 1.27 1.27)
+				)
+				(hide yes)
+			)
+		)
 		(pin "1"
 		)
@@
 			)
 		)
-		(property "Part URL" ""
+		(property "Part URL" "https://mou.sr/4aLzHIM"
 			(at 190.5 76.2 0)
 			(effects
@@
 			)
 		)
-		(property "Vendor" ""
+		(property "Vendor" "Mouser"
 			(at 190.5 76.2 0)
 			(effects
@@
 			)
 		)
+		(property "Part no." "603-MFR-25FRF5210K"
+			(at 190.5 76.2 0)
+			(effects
+				(font
+					(size 1.27 1.27)
+				)
+				(hide yes)
+			)
+		)
 		(pin "1"
 		)
@@
 			)
 		)
-		(property "Part URL" ""
+		(property "Part URL" "https://mou.sr/4kxE3Vr"
 			(at 139.7 166.37 0)
 			(effects
@@
 			)
 		)
-		(property "Vendor" ""
+		(property "Vendor" "Mouser"
 			(at 139.7 166.37 0)
 			(effects
@@
 			)
 		)
+		(property "Part no." "200-SSW10401TMS"
+			(at 139.7 166.37 0)
+			(effects
+				(font
+					(size 1.27 1.27)
+				)
+				(hide yes)
+			)
+		)
 		(pin "3"
 		)
@@
 			)
 		)
-		(property "Part URL" ""
+		(property "Part URL" "https://mou.sr/3PSKVAZ"
 			(at 106.68 80.01 0)
 			(effects
@@
 			)
 		)
-		(property "Vendor" ""
+		(property "Vendor" "Mouser"
 			(at 106.68 80.01 0)
 			(effects
@@
 			(at 106.68 80.01 0)
 			(effects
+				(font
+					(size 1.27 1.27)
+				)
+				(hide yes)
+			)
+		)
+		(property "Part no." "603-MFR-25FRF5220K"
+			(at 106.68 80.01 0)
+			(effects

Commit message: Fixed pot part number bug for Mixer module
Parts:
- RV_IN4, RV_IN4_GAIN1, RV_MAIN_VOL1, RV_THRESHOLD1: Part URL https://mou.sr/4694GMU -> https://mou.sr/47O2sTG; Part no. 652-PTV09A4025FB104 -> 652-PTV09A-4025UA104
Changed lines of the file:
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@@
 			)
 		)
-		(property "Part URL" "https://mou.sr/4694GMU"
+		(property "Part URL" "https://mou.sr/47O2sTG"
 			(at 106.68 88.9 0)
 			(effects
@@
 			)
 		)
-		(property "Part no." "652-PTV09A4025FB104"
+		(property "Part no." "652-PTV09A-4025UA104 "
 			(at 106.68 88.9 0)
 			(effects
@@
 			)
 		)
-		(property "Part URL" "https://mou.sr/4694GMU"
+		(property "Part URL" "https://mou.sr/47O2sTG"
 			(at 212.09 58.42 0)
 			(effects
@@
 			)
 		)
-		(property "Part no." "652-PTV09A4025FB104"
+		(property "Part no." "652-PTV09A-4025UA104 "
 			(at 212.09 58.42 0)
 			(effects
@@
 			)
 		)
-		(property "Part URL" "https://mou.sr/4694GMU"
+		(property "Part URL" "https://mou.sr/47O2sTG"
 			(at 106.68 57.15 0)
 			(effects
@@
 			)
 		)
-		(property "Part no." "652-PTV09A4025FB104"
+		(property "Part no." "652-PTV09A-4025UA104 "
 			(at 106.68 57.15 0)
 			(effects
@@
 			)
 		)
-		(property "Part URL" "https://mou.sr/4694GMU"
+		(property "Part URL" "https://mou.sr/47O2sTG"
 			(at 180.34 76.2 0)
 			(effects
@@
 			)
 		)
-		(property "Part no." "652-PTV09A4025FB104"
+		(property "Part no." "652-PTV09A-4025UA104 "
 			(at 180.34 76.2 0)
 			(effects

Commit message: Updated UI BOMs
Parts:
- RV_IN4, RV_IN4_GAIN1, RV_MAIN_VOL1, RV_THRESHOLD1: Note (none) -> Knurled Shaft

Commit message: Fixed socket to header on mixer UI
Parts:
- J3, J7: footprint Connector_PinHeader_2.54mm:PinHeader_1x04_P2.54mm_Vertical -> Connector_PinSocket_2.54mm:PinSocket_1x04_P2.54mm_Vertical
Changed lines of the file:
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@@
 			)
 		)
-		(property "Footprint" "Connector_PinHeader_2.54mm:PinHeader_1x04_P2.54mm_Vertical"
+		(property "Footprint" "Connector_PinSocket_2.54mm:PinSocket_1x04_P2.54mm_Vertical"
 			(at 139.7 148.59 0)
 			(effects
@@
 			)
 		)
-		(property "Footprint" "Connector_PinHeader_2.54mm:PinHeader_1x04_P2.54mm_Vertical"
+		(property "Footprint" "Connector_PinSocket_2.54mm:PinSocket_1x04_P2.54mm_Vertical"
 			(at 139.7 166.37 0)
 			(effects
