File: modules/06-utils-output/electronics/core/utils-output-core.kicad_sch (KiCad schematic)
At the start: 8 parts, among them J1 Conn_01x06, J4 Conn_02x04_Odd_Even, J5 Conn_02x03_Odd_Even, J6 Conn_02x05_Odd_Even

Commit message: Utils JLCPCB verified for v1.0
Parts:
- H1, H2, H3, H4, J4, J6: CHECKED YES -> (none)
- J5: Vendor (none) -> Mouser
Changed lines of the file:
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@@
 	(title_block
 		(title "Utils / Output")
-		(date "2025-10-24")
-		(rev "v0.2")
+		(date "2025-12-11")
+		(rev "v1.0")
 		(company "Shmøergh")
 	)
@@
 			)
 		)
-		(property "Vendor" ""
+		(property "Vendor" "Mouser"
 			(at 215.9 97.79 0)
 			(effects
@@
 			)
 		)
-		(property "CHECKED" "YES"
+		(property "CHECKED" ""
 			(at 200.66 160.02 0)
 			(effects
@@
 			)
 		)
-		(property "CHECKED" "YES"
+		(property "CHECKED" ""
 			(at 179.07 160.02 0)
 			(effects
@@
 			)
 		)
-		(property "CHECKED" "YES"
+		(property "CHECKED" ""
 			(at 215.9 121.92 0)
 			(effects
@@
 			)
 		)
-		(property "CHECKED" "YES"
+		(property "CHECKED" ""
 			(at 215.9 73.66 0)
 			(effects
@@
 			)
 		)
-		(property "CHECKED" "YES"
+		(property "CHECKED" ""
 			(at 220.98 160.02 0)
 			(effects
@@
 			)
 		)
-		(property "CHECKED" "YES"
+		(property "CHECKED" ""
 			(at 241.3 160.02 0)
 			(effects

Commit message: Added Utils BOM
Parts:
- J1: Mouser Part no. (none) -> 200-SSW10601TMS; Part URL (none) -> https://mou.sr/4puxA0F; Vendor (none) -> Mouser
- J4: Mouser Part no. (none) -> 200-HTSW10407TD; Part URL (none) -> https://mou.sr/4nYsZDt; Vendor (none) -> Mouser
- J5: Mouser Part no. (none) -> 200-TSW10307TD; Part URL (none) -> https://mou.sr/4liCQlU
- J6: Mouser Part no. (none) -> 200-TSW10507TD; Part URL (none) -> https://mou.sr/40QhDaC; Vendor (none) -> Mouser
Changed lines of the file:
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@@
 			)
 		)
-		(property "Part URL" ""
+		(property "Part URL" "https://mou.sr/4liCQlU"
 			(at 215.9 97.79 0)
 			(effects
@@
 		)
 		(property "LCSC" ""
+			(at 215.9 97.79 0)
+			(effects
+				(font
+					(size 1.27 1.27)
+				)
+				(hide yes)
+			)
+		)
+		(property "Mouser Part no." "200-TSW10307TD"
 			(at 215.9 97.79 0)
 			(effects
@@
 			)
 		)
-		(property "Part URL" ""
+		(property "Part URL" "https://mou.sr/4puxA0F"
 			(at 218.44 45.72 0)
 			(effects
@@
 			)
 		)
-		(property "Vendor" ""
+		(property "Vendor" "Mouser"
 			(at 218.44 45.72 0)
 			(effects
@@
 		)
 		(property "LCSC" ""
+			(at 218.44 45.72 0)
+			(effects
+				(font
+					(size 1.27 1.27)
+				)
+				(hide yes)
+			)
+		)
+		(property "Mouser Part no." "200-SSW10601TMS"
 			(at 218.44 45.72 0)
 			(effects
@@
 			)
 		)
-		(property "Part URL" ""
-			(at 215.9 121.92 0)
-			(effects
-				(font
-					(size 1.27 1.27)
-				)
-				(hide yes)
-			)
-		)
-		(property "Vendor" ""
+		(property "Part URL" "https://mou.sr/40QhDaC"
+			(at 215.9 121.92 0)
+			(effects
+				(font
+					(size 1.27 1.27)
+				)
+				(hide yes)
+			)
+		)
+		(property "Vendor" "Mouser"
 			(at 215.9 121.92 0)
 			(effects
@@
 		)
 		(property "CHECKED" ""
+			(at 215.9 121.92 0)
+			(effects
+				(font
+					(size 1.27 1.27)
+				)
+				(hide yes)
+			)
+		)
+		(property "Mouser Part no." "200-TSW10507TD"
 			(at 215.9 121.92 0)
 			(effects
@@
 			)
 		)
-		(property "Part URL" ""
-			(at 215.9 73.66 0)
-			(effects
-				(font
-					(size 1.27 1.27)
-				)
-				(hide yes)
-			)
-		)
-		(property "Vendor" ""
+		(property "Part URL" "https://mou.sr/4nYsZDt"
+			(at 215.9 73.66 0)
+			(effects
+				(font
+					(size 1.27 1.27)
+				)
+				(hide yes)
+			)
+		)
+		(property "Vendor" "Mouser"
 			(at 215.9 73.66 0)
 			(effects
@@
 			(at 215.9 73.66 0)
 			(effects
+				(font
+					(size 1.27 1.27)
+				)
+				(hide yes)
+			)
+		)
+		(property "Mouser Part no." "200-HTSW10407TD"
+			(at 215.9 73.66 0)
+			(effects

Commit message: Set Utils core default patch connector to DNP
Parts:
- J1: now not fitted
Changed lines of the file:
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@@
 		(in_bom yes)
 		(on_board yes)
-		(dnp no)
+		(dnp yes)
 		(fields_autoplaced yes)
 		(property "Reference" "J1"

Commit message: KiCAD version update - Utils
Other:
- title: Utils / Output -> Utils / Output Core
Changed lines of the file:
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@@
 	(paper "A4")
 	(title_block
-		(title "Utils / Output")
-		(date "2025-12-11")
-		(rev "v1.0")
+		(title "Utils / Output Core")
+		(date "2026-02-21")
+		(rev "v1.1")
 		(company "Shmøergh")
 	)
