File: modules/06-utils-output/electronics/core/sheets/bitcrusher-sh.kicad_sch (KiCad schematic)
At the start: 27 parts, among them Q2 2N3819, U1 TL072, U2 TL072

Commit message: Utils JLCPCB verified for v1.0
Parts:
- C16, C17, C18, Q2: CHECKED YES -> (none)
Changed lines of the file:
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@@
 			)
 		)
-		(property "CHECKED" "YES"
+		(property "CHECKED" ""
 			(at 179.07 55.88 0)
 			(effects
@@
 			)
 		)
-		(property "CHECKED" "YES"
+		(property "CHECKED" ""
 			(at 161.29 106.68 90)
 			(effects
@@
 			)
 		)
-		(property "CHECKED" "YES"
+		(property "CHECKED" ""
 			(at 69.85 110.49 0)
 			(effects
@@
 			)
 		)
-		(property "CHECKED" "YES"
+		(property "CHECKED" ""
 			(at 166.37 50.8 90)
 			(effects

Commit message: Added Utils BOM
Parts:
- C16, C17: CHECKED (none) -> YES; Mouser Part no. (none) -> 80-MMK5104J50J01L16; Part URL (none) -> https://mou.sr/4iTinUl; Vendor (none) -> Mouser
- C18: CHECKED (none) -> YES; Mouser Part no. (none) -> 80-MMK5102M50J01L4; Part URL (none) -> https://mou.sr/4rSWoRD; Vendor (none) -> Mouser
- Q2: Mouser Part no. (none) -> 610-2N3819; Part URL (none) -> https://mou.sr/4rVtQ9Z; Vendor (none) -> Mouser
Changed lines of the file:
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@@
 			)
 		)
-		(property "Part URL" ""
+		(property "Part URL" "https://mou.sr/4iTinUl"
 			(at 179.07 55.88 0)
 			(effects
@@
 			)
 		)
-		(property "Vendor" ""
+		(property "Vendor" "Mouser"
 			(at 179.07 55.88 0)
 			(effects
@@
 			)
 		)
-		(property "CHECKED" ""
+		(property "CHECKED" "YES"
+			(at 179.07 55.88 0)
+			(effects
+				(font
+					(size 1.27 1.27)
+				)
+				(hide yes)
+			)
+		)
+		(property "Mouser Part no." "80-MMK5104J50J01L16 "
 			(at 179.07 55.88 0)
 			(effects
@@
 			)
 		)
-		(property "Part URL" ""
+		(property "Part URL" "https://mou.sr/4rSWoRD"
 			(at 161.29 106.68 0)
 			(effects
@@
 			)
 		)
-		(property "Vendor" ""
+		(property "Vendor" "Mouser"
 			(at 161.29 106.68 0)
 			(effects
@@
 			)
 		)
-		(property "CHECKED" ""
+		(property "CHECKED" "YES"
+			(at 161.29 106.68 90)
+			(effects
+				(font
+					(size 1.27 1.27)
+				)
+				(hide yes)
+			)
+		)
+		(property "Mouser Part no." "80-MMK5102M50J01L4 "
 			(at 161.29 106.68 90)
 			(effects
@@
 			)
 		)
-		(property "Part URL" ""
+		(property "Part URL" "https://mou.sr/4iTinUl"
 			(at 69.85 110.49 0)
 			(effects
@@
 			)
 		)
-		(property "Vendor" ""
+		(property "Vendor" "Mouser"
 			(at 69.85 110.49 0)
 			(effects
@@
 			)
 		)
-		(property "CHECKED" ""
+		(property "CHECKED" "YES"
+			(at 69.85 110.49 0)
+			(effects
+				(font
+					(size 1.27 1.27)
+				)
+				(hide yes)
+			)
+		)
+		(property "Mouser Part no." "80-MMK5104J50J01L16 "
 			(at 69.85 110.49 0)
 			(effects
@@
 			)
 		)
-		(property "Part URL" ""
+		(property "Part URL" "https://mou.sr/4rVtQ9Z"
 			(at 166.37 50.8 0)
 			(effects
@@
 			)
 		)
-		(property "Vendor" ""
+		(property "Vendor" "Mouser"
 			(at 166.37 50.8 0)
 			(effects
@@
 			(at 166.37 50.8 90)
 			(effects
+				(font
+					(size 1.27 1.27)
+				)
+				(hide yes)
+			)
+		)
+		(property "Mouser Part no." "610-2N3819"
+			(at 166.37 50.8 90)
+			(effects

Commit message: KiCAD version update - Utils
Other:
- company: (none) -> Shmøergh
- title: (none) -> Utils / Output Core
Changed lines of the file:
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@@
 	(generator_version "9.0")
 	(paper "A4")
+	(title_block
+		(title "Utils / Output Core")
+		(date "2026-02-21")
+		(rev "v1.1")
+		(company "Shmøergh")
+	)
 	(rectangle
 		(start 82.55 132.08)
