File: modules/06-utils-output/electronics/core/sheets/lfo.kicad_sch (KiCad schematic)
At the start: 16 parts, among them U201 TL072

Commit message: Utils JLCPCB verified for v1.0
Parts:
- C203, R206: CHECKED YES -> (none)
- R203: LCSC C25811 -> C22809
- R207: LCSC C22962 -> C22790
- R210: LCSC C25811 -> C22975
- R211: LCSC C22962 -> C25804
Changed lines of the file:
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@@
 			)
 		)
-		(property "LCSC" "C25811"
+		(property "LCSC" "C22975"
 			(at 191.77 96.52 90)
 			(effects
@@
 			)
 		)
-		(property "LCSC" "C22962"
+		(property "LCSC" "C22790"
 			(at 134.62 77.47 90)
 			(effects
@@
 			)
 		)
-		(property "CHECKED" "YES"
+		(property "CHECKED" ""
 			(at 128.27 111.76 0)
 			(effects
@@
 			)
 		)
-		(property "CHECKED" "YES"
+		(property "CHECKED" ""
 			(at 171.45 111.76 90)
 			(effects
@@
 			)
 		)
-		(property "LCSC" "C25811"
+		(property "LCSC" "C22809"
 			(at 125.73 68.58 90)
 			(effects
@@
 			)
 		)
-		(property "LCSC" "C22962"
+		(property "LCSC" "C25804"
 			(at 200.66 105.41 90)
 			(effects

Commit message: Added Utils BOM
Parts:
- C203: CHECKED (none) -> YES]; Mouser Part no. (none) -> 80-R82EC1330AA50K
- R206: Mouser Part no. (none) -> 603-MFR-25FTF52-220R; Part URL (none) -> https://mou.sr/3XROtWU; Vendor (none) -> Mouser
Changed lines of the file:
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@@
 			)
 		)
-		(property "Part URL" ""
-			(at 128.27 111.76 0)
-			(effects
-				(font
-					(size 1.27 1.27)
-				)
-				(hide yes)
-			)
-		)
-		(property "Vendor" ""
+		(property "Part URL" "https://mou.sr/3XROtWU"
+			(at 128.27 111.76 0)
+			(effects
+				(font
+					(size 1.27 1.27)
+				)
+				(hide yes)
+			)
+		)
+		(property "Vendor" "Mouser"
 			(at 128.27 111.76 0)
 			(effects
@@
 		)
 		(property "CHECKED" ""
+			(at 128.27 111.76 0)
+			(effects
+				(font
+					(size 1.27 1.27)
+				)
+				(hide yes)
+			)
+		)
+		(property "Mouser Part no." "603-MFR-25FTF52-220R "
 			(at 128.27 111.76 0)
 			(effects
@@
 			)
 		)
-		(property "CHECKED" ""
+		(property "CHECKED" "YES]"
 			(at 171.45 111.76 90)
 			(effects
+				(font
+					(size 1.27 1.27)
+				)
+				(hide yes)
+			)
+		)
+		(property "Mouser Part no." "80-R82EC1330AA50K "
+			(at 171.45 111.76 90)
+			(effects

Commit message: KiCAD version update - Utils
Other:
- company: (none) -> Shmøergh
- title: (none) -> Utils / Output Core
Changed lines of the file:
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@@
 	(generator_version "9.0")
 	(paper "A4")
+	(title_block
+		(title "Utils / Output Core")
+		(date "2026-02-21")
+		(rev "v1.1")
+		(company "Shmøergh")
+	)
 	(text "Pot: A500k"
 		(exclude_from_sim no)
