File: modules/06-utils-output/electronics/core/sheets/power.kicad_sch (KiCad schematic)
At the start: 7 parts, among them J2 Conn_02x03_Odd_Even, J3 Conn_01x02, J7 Conn_02x05_Odd_Even

Commit message: Utils JLCPCB verified for v1.0
Parts:
- J2, J3, J7: CHECKED YES -> (none)
Changed lines of the file:
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@@
 			)
 		)
-		(property "CHECKED" "YES"
+		(property "CHECKED" ""
 			(at 88.9 92.71 0)
 			(effects
@@
 			)
 		)
-		(property "CHECKED" "YES"
+		(property "CHECKED" ""
 			(at 156.21 97.79 0)
 			(effects
@@
 			)
 		)
-		(property "CHECKED" "YES"
+		(property "CHECKED" ""
 			(at 92.71 109.22 0)
 			(effects

Commit message: Added Utils BOM
Parts:
- J2: Mouser Part no. (none) -> 200-TSW10307TD; Part URL (none) -> https://mou.sr/4liCQlU
- J3: Mouser Part no. (none) -> 200-HTSW10207TS; Part URL (none) -> https://mou.sr/3IruU3e
- J7: Mouser Part no. (none) -> 571-5103310-1; Part URL (none) -> https://mou.sr/3GwYxj9
Changed lines of the file:
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@@
 			)
 		)
-		(property "Part URL" ""
+		(property "Part URL" "https://mou.sr/4liCQlU"
 			(at 88.9 92.71 0)
 			(effects
@@
 			)
 		)
-		(property "Mouser Part no." ""
+		(property "Mouser Part no." "200-TSW10307TD"
 			(at 88.9 92.71 0)
 			(effects
@@
 			)
 		)
-		(property "Part URL" ""
+		(property "Part URL" "https://mou.sr/3GwYxj9"
 			(at 156.21 97.79 0)
 			(effects
@@
 			)
 		)
-		(property "Mouser Part no." ""
+		(property "Mouser Part no." "571-5103310-1"
 			(at 156.21 97.79 0)
 			(effects
@@
 			)
 		)
-		(property "Part URL" ""
+		(property "Part URL" "https://mou.sr/3IruU3e"
 			(at 92.71 109.22 0)
 			(effects
@@
 			)
 		)
-		(property "Mouser Part no." ""
+		(property "Mouser Part no." "200-HTSW10207TS"
 			(at 92.71 109.22 0)
 			(effects

Commit message: Updated out-of-stock 100uF cap JLCPCB product no's
Parts:
- C8, C9: LCSC C2836437 -> C2836442
Changed lines of the file:
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@@
 			)
 		)
-		(property "LCSC" "C2836437"
+		(property "LCSC" "C2836442"
 			(at 231.14 91.44 0)
 			(effects
@@
 			)
 		)
-		(property "LCSC" "C2836437"
+		(property "LCSC" "C2836442"
 			(at 231.14 99.06 0)
 			(effects

Commit message: KiCAD version update - Utils
Other:
- company: (none) -> Shmøergh
- title: (none) -> Utils / Output Core
Changed lines of the file:
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@@
 	(generator_version "9.0")
 	(paper "A4")
+	(title_block
+		(title "Utils / Output Core")
+		(date "2026-02-21")
+		(rev "v1.1")
+		(company "Shmøergh")
+	)
 	(text "UI power connection"
 		(exclude_from_sim no)
