File: modules/06-utils-output/experimental/ui-l+r-out/utils-output-ui.kicad_pcb (KiCad board)
At the start: 2 copper layers, 58 x 110 mm, 49 parts, among them J1 Conn_02x03_Odd_Even, J2 Conn_02x04_Odd_Even, J3 Conn_01x01_Pin, J4 Conn_01x02, J5 Conn_01x06, J6 Conn_02x05_Odd_Even, J7 Conn_02x03_Odd_Even, J8 Conn_01x01_Pin, Q1 2N3904, Q2 2N3906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

Commit message: Changed board versioning to 'rev' on Utils
Other:
- board text added: "UTILS+OUTPUT REV 3"
- board text removed: "SM-06 UTILS+OUTPUT V1.2"

Commit message: Fixed Utils experimental UI schemo and PCB after fckckin KiCAD update
Other:
- board text added: "UTILS+OUTPUT REV 4"
- board text removed: "UTILS+OUTPUT REV 3"
