File: modules/07-brain/electronics/core/sheets/audio-cv-in.kicad_sch (KiCad schematic)
At the start: 20 parts, among them U8 TL072, U9 TL072

Commit message: KiCAD version update - Brain
Other:
- company: (none) -> Shmøergh
- title: (none) -> Brain Core
Changed lines of the file:
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@@
 	(generator_version "9.0")
 	(paper "A4")
+	(title_block
+		(title "Brain Core")
+		(date "2026-02-21")
+		(rev "v1.1")
+		(company "Shmøergh")
+	)
 	(junction
 		(at 149.86 111.76)
