File: modules/07-brain/electronics/core/sheets/pots.kicad_sch (KiCad schematic)
At the start: 3 parts, among them U10 74HC4051

Commit message: KiCAD version update - Brain
Other:
- company: (none) -> Shmøergh
- title: (none) -> Brain Core
Changed lines of the file:
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@@
 	(generator_version "9.0")
 	(paper "A4")
+	(title_block
+		(title "Brain Core")
+		(date "2026-02-21")
+		(rev "v1.1")
+		(company "Shmøergh")
+	)
 	(rectangle
 		(start 57.15 50.8)
