File: modules/07-brain/electronics/core/sheets/pulse-io.kicad_sch (KiCad schematic)
At the start: 6 parts, among them Q1 MMBT3904, Q3 MMBT3904

Commit message: Added protection resistor to pulse out on Brain
Parts:
- added R13: 1k, Resistor_SMD:R_0603_1608Metric, symbol Device:R
Connections:
- net PULSE_OUT: now also R13.2; no longer Q3.3 (C), R3.1, R4.2
- new net: Q3.3 (C), R13.1, R3.1, R4.2
Other:
- note added: "About 5V pulses"
- note removed: "About 5.1V pulses"
Changed lines of the file:
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@@
 	(generator_version "9.0")
 	(paper "A4")
-	(text "About 5.1V pulses"
+	(text "About 5V pulses"
 		(exclude_from_sim no)
-		(at 209.55 77.47 0)
+		(at 208.28 71.12 0)
 		(effects
 			(font
@@
 	(wire
 		(pts
+			(xy 224.79 80.01) (xy 228.6 80.01)
+		)
+		(stroke
+			(width 0)
+			(type default)
+		)
+	)
+	(wire
+		(pts
 			(xy 209.55 83.82) (xy 209.55 80.01)
 		)
@@
 	(wire
 		(pts
-			(xy 209.55 80.01) (xy 215.9 80.01)
+			(xy 209.55 80.01) (xy 217.17 80.01)
 		)
 		(stroke
@@
 	(hierarchical_label "PULSE_OUT"
 		(shape output)
-		(at 215.9 80.01 0)
+		(at 228.6 80.01 0)
 		(effects
 			(font
@@
 		)
 	)
+	(symbol
+		(lib_id "Device:R")
+		(at 220.98 80.01 90)
+		(mirror x)
+		(unit 1)
+		(exclude_from_sim no)
+		(in_bom yes)
+		(on_board yes)
+		(dnp no)
+		(property "Reference" "R13"
+			(at 220.98 77.47 90)
+			(effects
+				(font
+					(size 1.27 1.27)
+				)
+			)
+		)
+		(property "Value" "1k"
+			(at 220.98 74.93 90)
+			(effects
+				(font
+					(size 1.27 1.27)
+				)
+			)
+		)
+		(property "Footprint" "Resistor_SMD:R_0603_1608Metric"
+			(at 220.98 78.232 90)
+			(effects
+				(font
+					(size 1.27 1.27)
+				)
+				(hide yes)
+			)
+		)
+		(property "Datasheet" "~"
+			(at 220.98 80.01 0)
+			(effects
+				(font
+					(size 1.27 1.27)
+				)
+				(hide yes)
+			)
+		)
+		(property "Description" ""
+			(at 220.98 80.01 0)
+			(effects
+				(font
+					(size 1.27 1.27)
+				)
+				(hide yes)
+			)
+		)
+		(property "LCSC" "C21190"
+			(at 220.98 80.01 90)
+			(effects
+				(font
+					(size 1.27 1.27)
+				)
+				(hide yes)
+			)
+		)
+		(property "Mouser" ""
+			(at 220.98 80.01 0)
+			(effects
+				(font
+					(size 1.27 1.27)
+				)
+				(hide yes)
+			)
+		)
+		(property "Part No." ""
+			(at 220.98 80.01 0)
+			(effects
+				(font
+					(size 1.27 1.27)
+				)
+				(hide yes)
+			)
+		)
+		(property "Part URL" ""
+			(at 220.98 80.01 0)
+			(effects
+				(font
+					(size 1.27 1.27)
+				)
+				(hide yes)
+			)
+		)
+		(property "Vendor" "JLCPCB"
+			(at 220.98 80.01 0)
+			(effects
+				(font
+					(size 1.27 1.27)
+				)
+				(hide yes)
+			)
+		)
+		(property "Field4" ""
+			(at 220.98 80.01 0)
+			(effects
+				(font
+					(size 1.27 1.27)
+				)
+				(hide yes)
+			)
+		)
+		(property "Sim.Device" ""
+			(at 220.98 80.01 90)
+			(effects
+				(font
+					(size 1.27 1.27)
+				)
+				(hide yes)
+			)
+		)
+		(property "Sim.Pins" ""
+			(at 220.98 80.01 90)
+			(effects
+				(font
+					(size 1.27 1.27)
+				)
+				(hide yes)
+			)
+		)
+		(property "CHECKED" "YES"
+			(at 220.98 80.01 90)
+			(effects
+				(font
+					(size 1.27 1.27)
+				)
+				(hide yes)
+			)
+		)
+		(pin "1"
+		)
+		(pin "2"
+		)
+		(instances
+			(project "brain-core"
+				(path "/8e2e31f3-eed5-4de1-966c-f4162758c735/b082d257-9358-41e3-a203-3f08ae6b6f5f"
+					(reference "R13")
+					(unit 1)
+				)
+			)
+		)
+	)

Commit message: KiCAD version update - Brain
Other:
- company: (none) -> Shmøergh
- title: (none) -> Brain Core
Changed lines of the file:
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@@
 	(generator_version "9.0")
 	(paper "A4")
+	(title_block
+		(title "Brain Core")
+		(date "2026-02-21")
+		(rev "v1.1")
+		(company "Shmøergh")
+	)
 	(text "About 5V pulses"
 		(exclude_from_sim no)
