File: modules/08-default-patch/default-patch.kicad_pcb (KiCad board)
At the start: 2 copper layers, 210.7 x 32.5 mm, 30 parts

Commit message: Default patch JLCPCB verified
Parts:
- moved G*** 4.89 mm to (66.2, 88.0)
Other:
- outline, holes or cut-outs redrawn
- board text added: "DEFAULT PATCH V1.0 - 2025"
- board text added: "DEFAULT PATCH V1.0 – 2025"
- board text removed: "DEFAULT PATCH V0.1 - 2025.12"
- board text removed: "DEFAULT PATCH V0.1 – 2025"
Changed lines of the file:
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@@
 		(locked yes)
 		(layer "F.Cu")
-		(at 66.477 83.114)
+		(at 66.223 88)
 		(property "Reference" "G***"
 			(at 0 0 0)
@@
 	)
 	(gr_arc
+		(start 71 83)
+		(mid 70.707107 83.707107)
+		(end 70 84)
+		(stroke
+			(width 0.05)
+			(type default)
+		)
+		(layer "Edge.Cuts")
+	)
+	(gr_arc
+		(start 60 85)
+		(mid 60.292893 84.292893)
+		(end 61 84)
+		(stroke
+			(width 0.05)
+			(type default)
+		)
+		(layer "Edge.Cuts")
+	)
+	(gr_arc
 		(start 63 92.5)
 		(mid 60.87868 91.62132)
@@
 	)
 	(gr_line
-		(start 60 79.5)
+		(start 60 85)
 		(end 60 89.5)
 		(stroke
@@
 	(gr_line
 		(start 60 63)
-		(end 60 70.5)
+		(end 60 68)
 		(stroke
 			(width 0.05)
@@
 		(layer "Edge.Cuts")
 	)
-	(gr_arc
-		(start 60 70.5)
-		(mid 64.5 75)
-		(end 60 79.5)
+	(gr_line
+		(start 70 84)
+		(end 61 84)
+		(stroke
+			(width 0.05)
+			(type default)
+		)
+		(layer "Edge.Cuts")
+	)
+	(gr_line
+		(start 61 69)
+		(end 70 69)
+		(stroke
+			(width 0.05)
+			(type default)
+		)
+		(layer "Edge.Cuts")
+	)
+	(gr_line
+		(start 71 70)
+		(end 71 83)
 		(stroke
 			(width 0.05)
@@
 		(layer "Edge.Cuts")
 	)
+	(gr_arc
+		(start 61 69)
+		(mid 60.292893 68.707107)
+		(end 60 68)
+		(stroke
+			(width 0.05)
+			(type default)
+		)
+		(layer "Edge.Cuts")
+	)
 	(gr_line
 		(start 267.7 92.5)
@@
 		(layer "Edge.Cuts")
 	)
+	(gr_arc
+		(start 70 69)
+		(mid 70.707107 69.292893)
+		(end 71 70)
+		(stroke
+			(width 0.05)
+			(type default)
+		)
+		(layer "Edge.Cuts")
+	)
 	(gr_text "GATE"
 		(at 76.637 84.892 90)
@@
 	)
 	(gr_text "SYNC"
-		(at 63.556 68.001 90)
+		(at 64.318 68.636 0)
 		(layer "F.SilkS")
 		(effects
@@
 	)
 	(gr_text "FM"
-		(at 66.096 67.874 90)
+		(at 66.604 68.636 0)
 		(layer "F.SilkS")
 		(effects
@@
 	)
 	(gr_text "PWM"
-		(at 68.636 67.874 90)
+		(at 69.525 68.636 0)
 		(layer "F.SilkS")
 		(effects
 			(font
-				(size 1 1)
+				(size 1 0.75)
 				(thickness 0.1)
 			)
@@
 		)
 	)
-	(gr_text "DEFAULT PATCH V0.1 - 2025.12"
+	(gr_text "DEFAULT PATCH V1.0 - 2025"
 		(at 206.812 77.653 0)
 		(layer "F.SilkS")
@@
 			(justify left bottom)
 		)
-		(render_cache "DEFAULT PATCH V0.1 - 2025.12" 0
+		(render_cache "DEFAULT PATCH V1.0 - 2025" 0
 			(polygon
 				(pts
@@
 			(polygon
 				(pts
-					(xy 220.289564 76.592124) (xy 220.289564 77.355749) (xy 220.416815 77.355749) (xy 220.416815 77.101187)
-					(xy 220.544126 77.101187) (xy 220.544126 76.973936) (xy 220.416815 76.973936) (xy 220.416815 76.592124)
+					(xy 220.544126 76.719374) (xy 220.544126 77.355749) (xy 220.289564 77.355749) (xy 220.289564 77.483)
+					(xy 220.925939 77.483) (xy 220.925939 77.355749) (xy 220.671377 77.355749) (xy 220.671377 76.464812)
+					(xy 220.544126 76.464812) (xy 220.544126 76.592124) (xy 220.289564 76.592124) (xy 220.289564 76.719374)
 				)
 			)
 			(polygon
 				(pts
-					(xy 220.416815 77.355749) (xy 220.416815 77.483) (xy 220.798627 77.483) (xy 220.798627 77.355749)
+					(xy 221.434147 77.228498) (xy 221.434147 77.483) (xy 221.561398 77.483) (xy 221.561398 77.228498)
 				)
 			)
 			(polygon
 				(pts
-					(xy 220.416815 76.464812) (xy 220.416815 76.592124) (xy 220.798627 76.592124) (xy 220.798627 76.464812)
+					(xy 222.069606 76.592124) (xy 222.069606 77.355749) (xy 222.196856 77.355749) (xy 222.196856 77.101187)
+					(xy 222.324168 77.101187) (xy 222.324168 76.973936) (xy 222.196856 76.973936) (xy 222.196856 76.592124)
 				)
 			)
 			(polygon
 				(pts
-					(xy 220.798627 76.592124) (xy 220.798627 76.719374) (xy 220.671377 76.719374) (xy 220.671377 76.846686)
-					(xy 220.798627 76.846686) (xy 220.798627 77.355749) (xy 220.925939 77.355749) (xy 220.925939 76.592124)
+					(xy 222.196856 77.355749) (xy 222.196856 77.483) (xy 222.578669 77.483) (xy 222.578669 77.355749)
 				)
 			)
 			(polygon
 				(pts
-					(xy 220.544126 76.846686) (xy 220.544126 76.973936) (xy 220.671377 76.973936) (xy 220.671377 76.846686)
+					(xy 222.196856 76.464812) (xy 222.196856 76.592124) (xy 222.578669 76.592124) (xy 222.578669 76.464812)
 				)
 			)
 			(polygon
 				(pts
-					(xy 221.434147 77.228498) (xy 221.434147 77.483) (xy 221.561398 77.483) (xy 221.561398 77.228498)
+					(xy 222.578669 76.592124) (xy 222.578669 76.719374) (xy 222.451419 76.719374) (xy 222.451419 76.846686)
+					(xy 222.578669 76.846686) (xy 222.578669 77.355749) (xy 222.705981 77.355749) (xy 222.705981 76.592124)
 				)
 			)
 			(polygon
 				(pts
-					(xy 222.324168 76.719374) (xy 222.324168 77.355749) (xy 222.069606 77.355749) (xy 222.069606 77.483)
-					(xy 222.705981 77.483) (xy 222.705981 77.355749) (xy 222.451419 77.355749) (xy 222.451419 76.464812)
-					(xy 222.324168 76.464812) (xy 222.324168 76.592124) (xy 222.069606 76.592124) (xy 222.069606 76.719374)
+					(xy 222.324168 76.846686) (xy 222.324168 76.973936) (xy 222.451419 76.973936) (xy 222.451419 76.846686)
 				)
 			)
@@
 				)
 			)
-			(polygon
-				(pts
-					(xy 229.444336 77.228498) (xy 229.444336 77.483) (xy 229.571586 77.483) (xy 229.571586 77.228498)
-				)
-			)
-			(polygon
-				(pts
-					(xy 230.334356 76.719374) (xy 230.334356 77.355749) (xy 230.079794 77.355749) (xy 230.079794 77.483)
-					(xy 230.716169 77.483) (xy 230.716169 77.355749) (xy 230.461607 77.355749) (xy 230.461607 76.464812)
-					(xy 230.334356 76.464812) (xy 230.334356 76.592124) (xy 230.079794 76.592124) (xy 230.079794 76.719374)
-				)
-			)
-			(polygon
-				(pts
-					(xy 230.969815 77.228498) (xy 230.969815 77.483) (xy 231.60619 77.483) (xy 231.60619 77.355749)
-					(xy 231.097066 77.355749) (xy 231.097066 77.228498)
-				)
-			)
-			(polygon
-				(pts
-					(xy 231.478878 76.592124) (xy 231.478878 76.464812) (xy 231.097066 76.464812) (xy 231.097066 76.592124)
-				)
-			)
-			(polygon
-				(pts
-					(xy 231.478878 76.592124) (xy 231.478878 76.846686) (xy 231.60619 76.846686) (xy 231.60619 76.592124)
-				)
-			)
-			(polygon
-				(pts
-					(xy 231.097066 77.101187) (xy 231.097066 77.228498) (xy 231.224377 77.228498) (xy 231.224377 77.101187)
-				)
-			)
-			(polygon
-				(pts
-					(xy 230.969815 76.592124) (xy 230.969815 76.719374) (xy 231.097066 76.719374) (xy 231.097066 76.592124)
-				)
-			)
-			(polygon
-				(pts
-					(xy 231.351628 76.846686) (xy 231.351628 76.973936) (xy 231.478878 76.973936) (xy 231.478878 76.846686)
-				)
-			)
-			(polygon
-				(pts
-					(xy 231.224377 76.973936) (xy 231.224377 77.101187) (xy 231.351628 77.101187) (xy 231.351628 76.973936)
-				)
-			)
 		)
 	)
@@
 	)
 	(gr_text "CV"
-		(at 71.176 67.874 90)
+		(at 71.684 68.636 0)
 		(layer "F.SilkS")
 		(effects
@@
 		)
 	)
-	(gr_text "DEFAULT PATCH V0.1 – 2025"
+	(gr_text "DEFAULT PATCH V1.0 – 2025"
 		(at 248.087 79.939 0)
 		(layer "B.SilkS")
@@
 			(justify left bottom mirror)
 		)
-		(render_cache "DEFAULT PATCH V0.1 – 2025" 0
+		(render_cache "DEFAULT PATCH V1.0 – 2025" 0
 			(polygon
 				(pts
@@
 			(polygon
 				(pts
-					(xy 234.609435 78.878124) (xy 234.609435 79.641749) (xy 234.482184 79.641749) (xy 234.482184 79.387187)
-					(xy 234.354873 79.387187) (xy 234.354873 79.259936) (xy 234.482184 79.259936) (xy 234.482184 78.878124)
+					(xy 234.354873 79.005374) (xy 234.354873 79.641749) (xy 234.609435 79.641749) (xy 234.609435 79.769)
+					(xy 233.97306 79.769) (xy 233.97306 79.641749) (xy 234.227622 79.641749) (xy 234.227622 78.750812)
+					(xy 234.354873 78.750812) (xy 234.354873 78.878124) (xy 234.609435 78.878124) (xy 234.609435 79.005374)
 				)
 			)
 			(polygon
 				(pts
-					(xy 234.482184 79.641749) (xy 234.482184 79.769) (xy 234.100372 79.769) (xy 234.100372 79.641749)
+					(xy 233.464852 79.514498) (xy 233.464852 79.769) (xy 233.337601 79.769) (xy 233.337601 79.514498)
 				)
 			)
 			(polygon
 				(pts
-					(xy 234.482184 78.750812) (xy 234.482184 78.878124) (xy 234.100372 78.878124) (xy 234.100372 78.750812)
+					(xy 232.829393 78.878124) (xy 232.829393 79.641749) (xy 232.702143 79.641749) (xy 232.702143 79.387187)
+					(xy 232.574831 79.387187) (xy 232.574831 79.259936) (xy 232.702143 79.259936) (xy 232.702143 78.878124)
 				)
 			)
 			(polygon
 				(pts
-					(xy 234.100372 78.878124) (xy 234.100372 79.005374) (xy 234.227622 79.005374) (xy 234.227622 79.132686)
-					(xy 234.100372 79.132686) (xy 234.100372 79.641749) (xy 233.97306 79.641749) (xy 233.97306 78.878124)
+					(xy 232.702143 79.641749) (xy 232.702143 79.769) (xy 232.32033 79.769) (xy 232.32033 79.641749)
 				)
 			)
 			(polygon
 				(pts
-					(xy 234.354873 79.132686) (xy 234.354873 79.259936) (xy 234.227622 79.259936) (xy 234.227622 79.132686)
+					(xy 232.702143 78.750812) (xy 232.702143 78.878124) (xy 232.32033 78.878124) (xy 232.32033 78.750812)
 				)
 			)
 			(polygon
 				(pts
-					(xy 233.464852 79.514498) (xy 233.464852 79.769) (xy 233.337601 79.769) (xy 233.337601 79.514498)
+					(xy 232.32033 78.878124) (xy 232.32033 79.005374) (xy 232.44758 79.005374) (xy 232.44758 79.132686)
+					(xy 232.32033 79.132686) (xy 232.32033 79.641749) (xy 232.193018 79.641749) (xy 232.193018 78.878124)
 				)
 			)
 			(polygon
 				(pts
-					(xy 232.574831 79.005374) (xy 232.574831 79.641749) (xy 232.829393 79.641749) (xy 232.829393 79.769)
-					(xy 232.193018 79.769) (xy 232.193018 79.641749) (xy 232.44758 79.641749) (xy 232.44758 78.750812)
-					(xy 232.574831 78.750812) (xy 232.574831 78.878124) (xy 232.829393 78.878124) (xy 232.829393 79.005374)
+					(xy 232.574831 79.132686) (xy 232.574831 79.259936) (xy 232.44758 79.259936) (xy 232.44758 79.132686)
 				)
 			)
@@
 	)
 	(gr_text "CV"
-		(at 70.033 68.001 270)
+		(at 69.779 68.636 0)
 		(layer "B.SilkS")
 		(effects
@@
 	)
 	(gr_text "SYNC"
-		(at 62.413 68.001 270)
+		(at 61.397 68.636 0)
 		(layer "B.SilkS")
 		(effects
@@
 	)
 	(gr_text "FM"
-		(at 64.953 68.001 270)
+		(at 64.445 68.636 0)
 		(layer "B.SilkS")
 		(effects
@@
 	)
 	(gr_text "PWM"
-		(at 67.493 68.001 270)
+		(at 66.985 68.636 0)
 		(layer "B.SilkS")
 		(effects
 			(font
-				(size 1 1)
+				(size 1 0.75)
 				(thickness 0.1)
 			)

Commit message: KiCAD version update - Default Patch
Other:
- board text added: "DEFAULT PATCH V1.0"
- board text removed: "DEFAULT PATCH V1.0 - 2025"
Changed lines of the file:
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@@
 		)
 	)
-	(gr_text "DEFAULT PATCH V1.0 - 2025"
+	(gr_text "DEFAULT PATCH V1.0"
 		(at 206.812 77.653 0)
 		(layer "F.SilkS")
@@
 			(justify left bottom)
 		)
-		(render_cache "DEFAULT PATCH V1.0 - 2025" 0
+		(render_cache "DEFAULT PATCH V1.0" 0
 			(polygon
 				(pts
@@
 				)
 			)
-			(polygon
-				(pts
-					(xy 224.358711 76.973936) (xy 223.976898 76.973936) (xy 223.976898 77.101187) (xy 224.358711 77.101187)
-				)
-			)
-			(polygon
-				(pts
-					(xy 225.62969 77.228498) (xy 225.62969 77.483) (xy 226.266064 77.483) (xy 226.266064 77.355749)
-					(xy 225.75694 77.355749) (xy 225.75694 77.228498)
-				)
-			)
-			(polygon
-				(pts
-					(xy 226.138753 76.592124) (xy 226.138753 76.464812) (xy 225.75694 76.464812) (xy 225.75694 76.592124)
-				)
-			)
-			(polygon
-				(pts
-					(xy 226.138753 76.592124) (xy 226.138753 76.846686) (xy 226.266064 76.846686) (xy 226.266064 76.592124)
-				)
-			)
-			(polygon
-				(pts
-					(xy 225.75694 77.101187) (xy 225.75694 77.228498) (xy 225.884252 77.228498) (xy 225.884252 77.101187)
-				)
-			)
-			(polygon
-				(pts
-					(xy 225.62969 76.592124) (xy 225.62969 76.719374) (xy 225.75694 76.719374) (xy 225.75694 76.592124)
-				)
-			)
-			(polygon
-				(pts
-					(xy 226.011502 76.846686) (xy 226.011502 76.973936) (xy 226.138753 76.973936) (xy 226.138753 76.846686)
-				)
-			)
-			(polygon
-				(pts
-					(xy 225.884252 76.973936) (xy 225.884252 77.101187) (xy 226.011502 77.101187) (xy 226.011502 76.973936)
-				)
-			)
-			(polygon
-				(pts
-					(xy 226.519711 76.592124) (xy 226.519711 77.355749) (xy 226.646961 77.355749) (xy 226.646961 77.101187)
-					(xy 226.774273 77.101187) (xy 226.774273 76.973936) (xy 226.646961 76.973936) (xy 226.646961 76.592124)
-				)
-			)
-			(polygon
-				(pts
-					(xy 226.646961 77.355749) (xy 226.646961 77.483) (xy 227.028774 77.483) (xy 227.028774 77.355749)
-				)
-			)
-			(polygon
-				(pts
-					(xy 226.646961 76.464812) (xy 226.646961 76.592124) (xy 227.028774 76.592124) (xy 227.028774 76.464812)
-				)
-			)
-			(polygon
-				(pts
-					(xy 227.028774 76.592124) (xy 227.028774 76.719374) (xy 226.901523 76.719374) (xy 226.901523 76.846686)
-					(xy 227.028774 76.846686) (xy 227.028774 77.355749) (xy 227.156085 77.355749) (xy 227.156085 76.592124)
-				)
-			)
-			(polygon
-				(pts
-					(xy 226.774273 76.846686) (xy 226.774273 76.973936) (xy 226.901523 76.973936) (xy 226.901523 76.846686)
-				)
-			)
-			(polygon
-				(pts
-					(xy 227.409732 77.228498) (xy 227.409732 77.483) (xy 228.046106 77.483) (xy 228.046106 77.355749)
-					(xy 227.536982 77.355749) (xy 227.536982 77.228498)
-				)
-			)
-			(polygon
-				(pts
-					(xy 227.918795 76.592124) (xy 227.918795 76.464812) (xy 227.536982 76.464812) (xy 227.536982 76.592124)
-				)
-			)
-			(polygon
-				(pts
-					(xy 227.918795 76.592124) (xy 227.918795 76.846686) (xy 228.046106 76.846686) (xy 228.046106 76.592124)
-				)
-			)
-			(polygon
-				(pts
-					(xy 227.536982 77.101187) (xy 227.536982 77.228498) (xy 227.664294 77.228498) (xy 227.664294 77.101187)
-				)
-			)
-			(polygon
-				(pts
-					(xy 227.409732 76.592124) (xy 227.409732 76.719374) (xy 227.536982 76.719374) (xy 227.536982 76.592124)
-				)
-			)
-			(polygon
-				(pts
-					(xy 227.791544 76.846686) (xy 227.791544 76.973936) (xy 227.918795 76.973936) (xy 227.918795 76.846686)
-				)
-			)
-			(polygon
-				(pts
-					(xy 227.664294 76.973936) (xy 227.664294 77.101187) (xy 227.791544 77.101187) (xy 227.791544 76.973936)
-				)
-			)
-			(polygon
-				(pts
-					(xy 228.299752 76.464812) (xy 228.299752 76.973936) (xy 228.808816 76.973936) (xy 228.808816 76.846686)
-					(xy 228.427003 76.846686) (xy 228.427003 76.592124) (xy 228.936127 76.592124) (xy 228.936127 76.464812)
-				)
-			)
-			(polygon
-				(pts
-					(xy 228.808816 76.973936) (xy 228.808816 77.355749) (xy 228.936127 77.355749) (xy 228.936127 76.973936)
-				)
-			)
-			(polygon
-				(pts
-					(xy 228.808816 77.355749) (xy 228.427003 77.355749) (xy 228.427003 77.483) (xy 228.808816 77.483)
-				)
-			)
-			(polygon
-				(pts
-					(xy 228.427003 77.355749) (xy 228.427003 77.228498) (xy 228.299752 77.228498) (xy 228.299752 77.355749)
-				)
-			)

Commit message: Changed board versioning to 'rev' on Default Patch
Other:
- board text added: "DEFAULT PATCH REV 1"
- board text removed: "DEFAULT PATCH V1.0"
- board text removed: "DEFAULT PATCH V1.0 – 2025"

Commit message: Fixed Default Patch schemo and PCB after fckckin KiCAD update
Other:
- board text added: "DEFAULT PATCH"
- board text added: "DEFAULT PATCH REV 2"
- board text removed: "DEFAULT PATCH REV 1"
